File: moco-o/braking_circuitkicad_sch.kicad_sch (KiCad schematic)
At the start: 14 parts, among them Q10 CSD18540Q5B, Q9 CSD18540Q5B, U6 LM5109A

Commit message: Move files
Changed lines of the file:
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@@
   )
   (symbol (lib_id "Driver_FET:LM5109MA") (at 115.57 77.47 0) (unit 1)
-    (in_bom yes) (on_board yes) (fields_autoplaced)
-    (property "Reference" "U6" (id 0) (at 115.57 62.23 0))
-    (property "Value" "LM5109A" (id 1) (at 115.57 64.77 0))
+    (in_bom yes) (on_board yes)
+    (property "Reference" "U6" (id 0) (at 115.57 63.5 0))
+    (property "Value" "LM5109A" (id 1) (at 115.57 66.04 0))
     (property "Footprint" "Package_SO:SOIC-8_3.9x4.9mm_P1.27mm" (id 2) (at 115.57 90.17 0)
       (effects (font (size 1.27 1.27) italic) hide)
