File: moco-o/mcu.kicad_sch (KiCad schematic)
At the start: 14 parts, among them U3 8MHz, U4 STM32F405RGTx

Commit message: Move files
Other:
- note removed: "Output current sunk/source by any I/Os and control pin is 25mA MAX"
- moved on the sheet: C39, C40, C41, C42, C43, C44, C45, C46, C47, C48, C49, C50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
