File: moco-o/moco.kicad_sch (KiCad schematic)
At the start: 93 parts, among them J1 USB_C_Receptacle_USB2.0, J2 Conn_02x10_Odd_Even, J3 Conn_01x02, J4 Conn_01x05, J5 SWD 10-Pin, J6 ST-LINK, J7 Conn_02x02_Odd_Even, J8 Conn_01x06, J9 Conn_01x06, Q1 AO3413, Q2 AO3413, SW1 SW_Push, SW2 SW_Push, SW3 SW_Push, SW4 SW_Push, U1 AMS1117-3.3

Commit message: Move files
Parts:
- removed J7: Conn_02x02_Odd_Even, Connector_PinHeader_2.54mm:PinHeader_2x02_P2.54mm_Horizontal, symbol Connector_Generic:Conn_02x02_Odd_Even
- added SB22: SolderJumper_2_Bridged, Jumper:SolderJumper-2_P1.3mm_Bridged_RoundedPad1.0x1.5mm, symbol Jumper:SolderJumper_2_Bridged
- J2: footprint Connector_PinHeader_2.54mm:PinHeader_2x10_P2.54mm_Horizontal -> Connector_PinHeader_2.54mm:PinHeader_2x08_P2.54mm_Vertical; symbol Connector_Generic:Conn_02x10_Odd_Even -> Connector_Generic:Conn_02x08_Odd_Even
- J3: footprint Connector_AMASS:AMASS_XT60-F_1x02_P7.20mm_Vertical -> Connector_AMASS:AMASS_XT60-M_1x02_P7.20mm_Vertical
- J4: footprint Connector_JST:JST_PH_S5B-PH-SM4-TB_1x05-1MP_P2.00mm_Horizontal -> Connector_JST:JST_GH_SM05B-GHS-TB_1x05-1MP_P1.25mm_Horizontal
- J6: footprint Connector_PinHeader_2.54mm:PinHeader_1x06_P2.54mm_Vertical -> Connector_PinHeader_2.54mm:PinHeader_1x05_P2.54mm_Vertical; symbol Connector_Generic:Conn_01x06 -> Connector_Generic:Conn_01x05
- J8: footprint Connector_JST:JST_PH_S6B-PH-SM4-TB_1x06-1MP_P2.00mm_Horizontal -> Connector_JST:JST_GH_SM06B-GHS-TB_1x06-1MP_P1.25mm_Horizontal
- J9: footprint Connector_JST:JST_PH_S6B-PH-SM4-TB_1x06-1MP_P2.00mm_Horizontal -> Connector_JST:JST_GH_BM06B-GHS-TBT_1x06-1MP_P1.25mm_Vertical
- JP1: footprint Connector_PinHeader_2.54mm:PinHeader_1x03_P2.54mm_Vertical -> Connector_PinHeader_2.54mm:PinHeader_1x03_P2.54mm_Vertical_SMD_Pin1Left; Note (none) -> Default 1-2 closed, 3 open
Connections:
- net GND: now also J2.15 (Pin_15), J2.16 (Pin_16); no longer J2.19 (Pin_19), J2.20 (Pin_20), J2.5 (Pin_5), J2.6 (Pin_6)
- net MCU_~{RESET}: no longer J2.3 (Pin_3)
- net PA0_CONN: now also J2.3 (Pin_3); no longer J2.7 (Pin_7)
- net PA15_CONN: now also J2.8 (Pin_8); no longer J2.12 (Pin_12)
- net PA1_CONN: now also J2.4 (Pin_4); no longer J2.8 (Pin_8)
- net PA2: now also J2.5 (Pin_5); no longer J2.9 (Pin_9)
- net PA3: now also J2.6 (Pin_6); no longer J2.10 (Pin_10)
- net PA7: now also J2.7 (Pin_7); no longer J2.11 (Pin_11)
- net PB0: now also J2.9 (Pin_9); no longer J2.13 (Pin_13)
- net PB1: now also J2.10 (Pin_10); no longer J2.14 (Pin_14)
- net PB2_CONN: now also J2.11 (Pin_11); no longer J2.15 (Pin_15)
- net PB3_CONN: now also J2.12 (Pin_12); no longer J2.16 (Pin_16)
- net PC4: now also J2.13 (Pin_13); no longer J2.17 (Pin_17)
- net PC8: now also J2.14 (Pin_14); no longer J2.18 (Pin_18)
- net VCC: now also SB5.1 (A), SB6.1 (A), SB22.2 (B); no longer J2.4 (Pin_4), Q1.2 (S), Q2.2 (S), R10.2, R26.1, R27.1, R28.1, R9.2
- net ~{FAULT}: now also R7.2; no longer SB5.2 (B)
- net ~{OCTW}: now also R8.2; no longer SB6.2 (B)
- new net: R26.1, R27.1, R28.1, SB22.1 (A)
- new net: Q2.2 (S), R10.2, SB5.2 (B)
- new net: Q1.2 (S), R9.2, SB6.2 (B)
- no-connect marks 7 -> 6
Other:
- title: (none) -> MoCo-O
- moved on the sheet: LD4, LD5, Q1, Q2, R10, R15, R16, R7, R8, R9
