File: moco-o/motor_driver.kicad_sch (KiCad schematic)
At the start: 66 parts, among them Q3 CSD18540Q5B, Q4 CSD18540Q5B, Q5 CSD18540Q5B, Q6 CSD18540Q5B, Q7 CSD18540Q5B, Q8 CSD18540Q5B, U2 DRV8301

Commit message: Move files
Parts:
- C31: footprint Capacitor_Tantalum_SMD:CP_EIA-7343-31_Kemet-D -> Capacitor_Tantalum_SMD:CP_EIA-6032-28_Kemet-C; JLCPCB Part # C11382 -> C7220; MFR.Part # TAJD686K016RNJ -> TAJC686K016RNJ
Changed lines of the file:
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@@
       (effects (font (size 1.27 1.27)) (justify left))
     )
-    (property "Footprint" "Capacitor_Tantalum_SMD:CP_EIA-7343-31_Kemet-D" (id 2) (at 166.0652 110.49 0)
+    (property "Footprint" "Capacitor_Tantalum_SMD:CP_EIA-6032-28_Kemet-C" (id 2) (at 166.0652 110.49 0)
       (effects (font (size 1.27 1.27)) hide)
     )
@@
       (effects (font (size 1.27 1.27)) hide)
     )
-    (property "JLCPCB Part #" "C11382" (id 4) (at 165.1 106.68 0)
+    (property "JLCPCB Part #" "C7220" (id 4) (at 165.1 106.68 0)
       (effects (font (size 1.27 1.27)) hide)
     )
-    (property "MFR.Part #" "TAJD686K016RNJ" (id 5) (at 165.1 106.68 0)
+    (property "MFR.Part #" "TAJC686K016RNJ" (id 5) (at 165.1 106.68 0)
       (effects (font (size 1.27 1.27)) hide)
     )
