File: moco-s/pos_sensor.kicad_sch (KiCad schematic)
At the start: 6 parts, among them U6 AS5147

Commit message: Comp MoCo-S
Parts:
- removed R12, R51: 10k, Resistor_SMD:R_0603_1608Metric, symbol Device:R
Other:
- moved on the sheet: R52
Changed lines of the file:
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@@
 (kicad_sch (version 20211123) (generator eeschema)
   (paper "A4")
+  (junction (at 134.62 99.06) (diameter 0) (color 0 0 0 0)
+  )
   (junction (at 162.56 111.76) (diameter 0) (color 0 0 0 0)
   )
-  (junction (at 105.41 91.44) (diameter 0) (color 0 0 0 0)
-  )
   (junction (at 162.56 72.39) (diameter 0) (color 0 0 0 0)
   )
   (junction (at 143.51 104.14) (diameter 0) (color 0 0 0 0)
   )
-  (junction (at 113.03 96.52) (diameter 0) (color 0 0 0 0)
-  )
-  (junction (at 119.38 99.06) (diameter 0) (color 0 0 0 0)
-  )
-  (wire (pts (xy 100.33 93.98) (xy 149.86 93.98))
-    (stroke (width 0) (type default) (color 0 0 0 0))
-  )
-  (wire (pts (xy 119.38 99.06) (xy 149.86 99.06))
+  (wire (pts (xy 125.73 93.98) (xy 149.86 93.98))
     (stroke (width 0) (type default) (color 0 0 0 0))
   )
@@
     (stroke (width 0) (type default) (color 0 0 0 0))
   )
-  (wire (pts (xy 100.33 96.52) (xy 113.03 96.52))
-    (stroke (width 0) (type default) (color 0 0 0 0))
-  )
-  (wire (pts (xy 105.41 91.44) (xy 105.41 101.6))
+  (wire (pts (xy 134.62 99.06) (xy 149.86 99.06))
     (stroke (width 0) (type default) (color 0 0 0 0))
   )
@@
     (stroke (width 0) (type default) (color 0 0 0 0))
   )
-  (wire (pts (xy 100.33 99.06) (xy 119.38 99.06))
+  (wire (pts (xy 125.73 99.06) (xy 134.62 99.06))
     (stroke (width 0) (type default) (color 0 0 0 0))
   )
@@
     (stroke (width 0) (type default) (color 0 0 0 0))
   )
-  (wire (pts (xy 100.33 91.44) (xy 105.41 91.44))
-    (stroke (width 0) (type default) (color 0 0 0 0))
-  )
   (wire (pts (xy 177.8 106.68) (xy 175.26 106.68))
     (stroke (width 0) (type default) (color 0 0 0 0))
   )
-  (wire (pts (xy 119.38 88.9) (xy 119.38 99.06))
+  (wire (pts (xy 134.62 88.9) (xy 134.62 99.06))
     (stroke (width 0) (type default) (color 0 0 0 0))
   )
@@
     (stroke (width 0) (type default) (color 0 0 0 0))
   )
-  (wire (pts (xy 113.03 96.52) (xy 113.03 101.6))
-    (stroke (width 0) (type default) (color 0 0 0 0))
-  )
-  (wire (pts (xy 105.41 91.44) (xy 149.86 91.44))
+  (wire (pts (xy 125.73 91.44) (xy 149.86 91.44))
     (stroke (width 0) (type default) (color 0 0 0 0))
   )
@@
     (stroke (width 0) (type default) (color 0 0 0 0))
   )
-  (wire (pts (xy 113.03 96.52) (xy 149.86 96.52))
+  (wire (pts (xy 125.73 96.52) (xy 149.86 96.52))
     (stroke (width 0) (type default) (color 0 0 0 0))
   )
@@
     (stroke (width 0) (type default) (color 0 0 0 0))
   )
-  (text "3.3V operation mode" (at 132.08 119.38 0)
+  (text "3.3V operation mode" (at 151.13 124.46 0)
     (effects (font (size 1.27 1.27)) (justify left bottom))
   )
-  (hierarchical_label "SPI_MISO" (shape output) (at 100.33 93.98 180)
+  (hierarchical_label "SPI_MISO" (shape output) (at 125.73 93.98 180)
     (effects (font (size 1.27 1.27)) (justify right))
   )
@@
     (effects (font (size 1.27 1.27)) (justify left))
   )
-  (hierarchical_label "SPI_CLK" (shape input) (at 100.33 96.52 180)
+  (hierarchical_label "SPI_CLK" (shape input) (at 125.73 96.52 180)
     (effects (font (size 1.27 1.27)) (justify right))
   )
@@
     (effects (font (size 1.27 1.27)) (justify left))
   )
-  (hierarchical_label "SPI_~{CS}" (shape input) (at 100.33 99.06 180)
+  (hierarchical_label "SPI_~{CS}" (shape input) (at 125.73 99.06 180)
     (effects (font (size 1.27 1.27)) (justify right))
   )
@@
     (effects (font (size 1.27 1.27)) (justify left))
   )
-  (hierarchical_label "SPI_MOSI" (shape input) (at 100.33 91.44 180)
+  (hierarchical_label "SPI_MOSI" (shape input) (at 125.73 91.44 180)
     (effects (font (size 1.27 1.27)) (justify right))
   )
@@
     (pin "1")
   )
-  (symbol (lib_id "Device:R") (at 105.41 105.41 0) (unit 1)
-    (in_bom yes) (on_board yes)
-    (property "Reference" "R12" (id 0) (at 106.68 104.14 0)
-      (effects (font (size 1.27 1.27)) (justify left))
-    )
-    (property "Value" "10k" (id 1) (at 106.68 106.68 0)
-      (effects (font (size 1.27 1.27)) (justify left))
-    )
-    (property "Footprint" "Resistor_SMD:R_0603_1608Metric" (id 2) (at 103.632 105.41 90)
-      (effects (font (size 1.27 1.27)) hide)
-    )
-    (property "Datasheet" "~" (id 3) (at 105.41 105.41 0)
-      (effects (font (size 1.27 1.27)) hide)
-    )
-    (property "JLCPCB Part #" "" (id 4) (at 105.41 105.41 0)
-      (effects (font (size 1.27 1.27)) hide)
-    )
-    (property "MFR.Part #" "" (id 5) (at 105.41 105.41 0)
-      (effects (font (size 1.27 1.27)) hide)
-    )
-    (pin "1")
-    (pin "2")
-  )
   (symbol (lib_id "power:GND") (at 162.56 111.76 0) (unit 1)
     (in_bom yes) (on_board yes)
@@
     (pin "2")
   )
-  (symbol (lib_id "Device:R") (at 119.38 85.09 0) (unit 1)
-    (in_bom yes) (on_board yes)
-    (property "Reference" "R52" (id 0) (at 120.65 83.82 0)
-      (effects (font (size 1.27 1.27)) (justify left))
-    )
-    (property "Value" "10k" (id 1) (at 120.65 86.36 0)
-      (effects (font (size 1.27 1.27)) (justify left))
-    )
-    (property "Footprint" "Resistor_SMD:R_0402_1005Metric" (id 2) (at 117.602 85.09 90)
-      (effects (font (size 1.27 1.27)) hide)
-    )
-    (property "Datasheet" "~" (id 3) (at 119.38 85.09 0)
-      (effects (font (size 1.27 1.27)) hide)
-    )
-    (property "JLCPCB Part #" "C25744" (id 4) (at 119.38 85.09 0)
-      (effects (font (size 1.27 1.27)) hide)
-    )
-    (property "MFR.Part #" "0402WGF1002TCE" (id 5) (at 119.38 85.09 0)
-      (effects (font (size 1.27 1.27)) hide)
-    )
-    (pin "1")
-    (pin "2")
-  )
-  (symbol (lib_id "power:GND") (at 105.41 109.22 0) (unit 1)
-    (in_bom yes) (on_board yes)
-    (property "Reference" "#PWR096" (id 0) (at 105.41 115.57 0)
-      (effects (font (size 1.27 1.27)) hide)
-    )
-    (property "Value" "GND" (id 1) (at 105.41 113.03 0))
-    (property "Footprint" "" (id 2) (at 105.41 109.22 0)
-      (effects (font (size 1.27 1.27)) hide)
-    )
-    (property "Datasheet" "" (id 3) (at 105.41 109.22 0)
-      (effects (font (size 1.27 1.27)) hide)
-    )
-    (pin "1")
-  )
-  (symbol (lib_id "power:VCC") (at 119.38 81.28 0) (unit 1)
-    (in_bom yes) (on_board yes)
-    (property "Reference" "#PWR098" (id 0) (at 119.38 85.09 0)
-      (effects (font (size 1.27 1.27)) hide)
-    )
-    (property "Value" "VCC" (id 1) (at 119.38 77.47 0))
-    (property "Footprint" "" (id 2) (at 119.38 81.28 0)
-      (effects (font (size 1.27 1.27)) hide)
-    )
-    (property "Datasheet" "" (id 3) (at 119.38 81.28 0)
-      (effects (font (size 1.27 1.27)) hide)
-    )
-    (pin "1")
-  )
-  (symbol (lib_id "power:GND") (at 113.03 109.22 0) (unit 1)
-    (in_bom yes) (on_board yes)
-    (property "Reference" "#PWR097" (id 0) (at 113.03 115.57 0)
-      (effects (font (size 1.27 1.27)) hide)
-    )
-    (property "Value" "GND" (id 1) (at 113.03 113.03 0))
-    (property "Footprint" "" (id 2) (at 113.03 109.22 0)
-      (effects (font (size 1.27 1.27)) hide)
-    )
-    (property "Datasheet" "" (id 3) (at 113.03 109.22 0)
+  (symbol (lib_id "Device:R") (at 134.62 85.09 0) (unit 1)
+    (in_bom yes) (on_board yes)
+    (property "Reference" "R52" (id 0) (at 135.89 83.82 0)
+      (effects (font (size 1.27 1.27)) (justify left))
+    )
+    (property "Value" "10k" (id 1) (at 135.89 86.36 0)
+      (effects (font (size 1.27 1.27)) (justify left))
+    )
+    (property "Footprint" "Resistor_SMD:R_0402_1005Metric" (id 2) (at 132.842 85.09 90)
+      (effects (font (size 1.27 1.27)) hide)
+    )
+    (property "Datasheet" "~" (id 3) (at 134.62 85.09 0)
+      (effects (font (size 1.27 1.27)) hide)
+    )
+    (property "JLCPCB Part #" "C25744" (id 4) (at 134.62 85.09 0)
+      (effects (font (size 1.27 1.27)) hide)
+    )
+    (property "MFR.Part #" "0402WGF1002TCE" (id 5) (at 134.62 85.09 0)
+      (effects (font (size 1.27 1.27)) hide)
+    )
+    (pin "1")
+    (pin "2")
+  )
+  (symbol (lib_id "power:VCC") (at 134.62 81.28 0) (unit 1)
+    (in_bom yes) (on_board yes)
+    (property "Reference" "#PWR098" (id 0) (at 134.62 85.09 0)
+      (effects (font (size 1.27 1.27)) hide)
+    )
+    (property "Value" "VCC" (id 1) (at 134.62 77.47 0))
+    (property "Footprint" "" (id 2) (at 134.62 81.28 0)
+      (effects (font (size 1.27 1.27)) hide)
+    )
+    (property "Datasheet" "" (id 3) (at 134.62 81.28 0)
       (effects (font (size 1.27 1.27)) hide)
     )
@@
     (pin "1")
   )
-  (symbol (lib_id "Device:R") (at 113.03 105.41 0) (unit 1)
-    (in_bom yes) (on_board yes)
-    (property "Reference" "R51" (id 0) (at 114.3 104.14 0)
-      (effects (font (size 1.27 1.27)) (justify left))
-    )
-    (property "Value" "10k" (id 1) (at 114.3 106.68 0)
-      (effects (font (size 1.27 1.27)) (justify left))
-    )
-    (property "Footprint" "Resistor_SMD:R_0603_1608Metric" (id 2) (at 111.252 105.41 90)
-      (effects (font (size 1.27 1.27)) hide)
-    )
-    (property "Datasheet" "~" (id 3) (at 113.03 105.41 0)
-      (effects (font (size 1.27 1.27)) hide)
-    )
-    (property "JLCPCB Part #" "" (id 4) (at 113.03 105.41 0)
-      (effects (font (size 1.27 1.27)) hide)
-    )
-    (property "MFR.Part #" "" (id 5) (at 113.03 105.41 0)
-      (effects (font (size 1.27 1.27)) hide)
-    )
-    (pin "1")
-    (pin "2")
-  )
   (symbol (lib_id "power:VCC") (at 138.43 104.14 90) (unit 1)

Commit message: Update ref
Parts:
- renumbered C54 to C49, C55 to C50, R52 to R38, U6 to U5
Changed lines of the file:
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@@
   (symbol (lib_id "Device:C") (at 156.21 76.2 0) (unit 1)
     (in_bom yes) (on_board yes)
-    (property "Reference" "C55" (id 0) (at 149.86 74.93 0)
+    (property "Reference" "C50" (id 0) (at 149.86 74.93 0)
       (effects (font (size 1.27 1.27)) (justify left))
     )
@@
   (symbol (lib_id "power:GND") (at 143.51 111.76 0) (unit 1)
     (in_bom yes) (on_board yes)
-    (property "Reference" "#PWR0100" (id 0) (at 143.51 118.11 0)
+    (property "Reference" "#PWR077" (id 0) (at 143.51 118.11 0)
       (effects (font (size 1.27 1.27)) hide)
     )
@@
   (symbol (lib_id "power:GND") (at 162.56 111.76 0) (unit 1)
     (in_bom yes) (on_board yes)
-    (property "Reference" "#PWR0103" (id 0) (at 162.56 118.11 0)
+    (property "Reference" "#PWR080" (id 0) (at 162.56 118.11 0)
       (effects (font (size 1.27 1.27)) hide)
     )
@@
   (symbol (lib_id "Device:C") (at 143.51 107.95 0) (unit 1)
     (in_bom yes) (on_board yes)
-    (property "Reference" "C54" (id 0) (at 137.16 106.68 0)
+    (property "Reference" "C49" (id 0) (at 137.16 106.68 0)
       (effects (font (size 1.27 1.27)) (justify left))
     )
@@
   (symbol (lib_id "Device:R") (at 134.62 85.09 0) (unit 1)
     (in_bom yes) (on_board yes)
-    (property "Reference" "R52" (id 0) (at 135.89 83.82 0)
+    (property "Reference" "R38" (id 0) (at 135.89 83.82 0)
       (effects (font (size 1.27 1.27)) (justify left))
     )
@@
   (symbol (lib_id "power:VCC") (at 134.62 81.28 0) (unit 1)
     (in_bom yes) (on_board yes)
-    (property "Reference" "#PWR098" (id 0) (at 134.62 85.09 0)
+    (property "Reference" "#PWR075" (id 0) (at 134.62 85.09 0)
       (effects (font (size 1.27 1.27)) hide)
     )
@@
   (symbol (lib_id "Sensor_Magnetic:AS5047D") (at 162.56 99.06 0) (unit 1)
     (in_bom yes) (on_board yes)
-    (property "Reference" "U6" (id 0) (at 166.37 83.82 0)
+    (property "Reference" "U5" (id 0) (at 166.37 83.82 0)
       (effects (font (size 1.27 1.27)) (justify left))
     )
@@
   (symbol (lib_id "power:VCC") (at 162.56 72.39 0) (unit 1)
     (in_bom yes) (on_board yes)
-    (property "Reference" "#PWR0102" (id 0) (at 162.56 76.2 0)
+    (property "Reference" "#PWR079" (id 0) (at 162.56 76.2 0)
       (effects (font (size 1.27 1.27)) hide)
     )
@@
   (symbol (lib_id "power:GND") (at 156.21 80.01 0) (unit 1)
     (in_bom yes) (on_board yes)
-    (property "Reference" "#PWR0101" (id 0) (at 156.21 86.36 0)
+    (property "Reference" "#PWR078" (id 0) (at 156.21 86.36 0)
       (effects (font (size 1.27 1.27)) hide)
     )
@@
   (symbol (lib_id "power:VCC") (at 138.43 104.14 90) (unit 1)
     (in_bom yes) (on_board yes)
-    (property "Reference" "#PWR099" (id 0) (at 142.24 104.14 0)
+    (property "Reference" "#PWR076" (id 0) (at 142.24 104.14 0)
       (effects (font (size 1.27 1.27)) hide)
     )

Commit message: Use kelvin connection for shunt resistance
Parts:
- U5: JLCPCB Part # (none) -> C481876; MFR.Part # AS5147 -> AS5147P-HTSM
Changed lines of the file:
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@@
       (effects (font (size 1.27 1.27)) hide)
     )
-    (property "JLCPCB Part #" "" (id 4) (at 162.56 99.06 0)
+    (property "JLCPCB Part #" "C481876" (id 4) (at 162.56 99.06 0)
       (effects (font (size 1.27 1.27)) hide)
     )
-    (property "MFR.Part #" "AS5147" (id 5) (at 162.56 99.06 0)
+    (property "MFR.Part #" "AS5147P-HTSM" (id 5) (at 162.56 99.06 0)
       (effects (font (size 1.27 1.27)) hide)
     )

Commit message: Replace some extended parts to basic parts
Parts:
- C49, C50, R38: Basic Part (none) -> Y
- U5: Basic Part (none) -> N
Changed lines of the file:
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@@
+      (effects (font (size 1.27 1.27)) hide)
+    )
+    (property "Basic Part" "Y" (id 6) (at 156.21 76.2 0)
       (effects (font (size 1.27 1.27)) hide)
     )
@@
       (effects (font (size 1.27 1.27)) hide)
     )
+    (property "Basic Part" "Y" (id 7) (at 143.51 107.95 0)
+      (effects (font (size 1.27 1.27)) hide)
+    )
     (pin "1")
     (pin "2")
@@
     )
     (property "MFR.Part #" "0402WGF1002TCE" (id 5) (at 134.62 85.09 0)
+      (effects (font (size 1.27 1.27)) hide)
+    )
+    (property "Basic Part" "Y" (id 6) (at 134.62 85.09 0)
       (effects (font (size 1.27 1.27)) hide)
     )
@@
       (effects (font (size 1.27 1.27)) hide)
     )
+    (property "Basic Part" "N" (id 6) (at 162.56 99.06 0)
+      (effects (font (size 1.27 1.27)) hide)
+    )
