File: moco-s/can_bus.kicad_sch (KiCad schematic)
At the start: 21 parts, among them J8 Conn_02x02_Top_Bottom, J9 Conn_02x02_Top_Bottom, U4 MCP2515-xST, U5 TJA1051T-3, Y3 8MHz

Commit message: Update layout
Parts:
- removed JP4, JP5: SolderJumper_3_Bridged12, Jumper:SolderJumper-3_P1.3mm_Bridged12_RoundedPad1.0x1.5mm_NumberLabels, symbol Jumper:SolderJumper_3_Bridged12
- removed SB21, SB22: SolderJumper_2_Bridged, Jumper:SolderJumper-2_P1.3mm_Bridged_RoundedPad1.0x1.5mm, symbol Jumper:SolderJumper_2_Bridged
- removed TP1, TP2: TestPoint, TestPoint:TestPoint_Pad_D2.0mm, symbol Connector:TestPoint
- C51: Note 47uF is better -> (none)
Connections:
- net MCP_RX is gone; now on net RX: U4.2 (RXCAN)
- net MCP_TX is gone; now on net TX: U4.1 (TXCAN)
- net ~{INT}: now reaches U4.13 (~{INT})
- net SPI_~{CS}: now reaches U4.18 (~{CS})
- net CAN_RX_TRN renamed RX
- net CAN_TX_TRN renamed TX
Other:
- moved on the sheet: C47, C48, C49, C50, C51, C52, C53, J8, J9, R47, R48, R49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

Commit message: Comp MoCo-S
Parts:
- removed C51: 10uF, Capacitor_Tantalum_SMD:CP_EIA-3216-18_Kemet-A, symbol Device:C_Polarized_Small
- removed C52: 100nF, Capacitor_SMD:C_0402_1005Metric, symbol Device:C_Small
- removed C53: 100pF, Capacitor_SMD:C_0402_1005Metric, symbol Device:C_Small
- removed R47, R48: 10k, Resistor_SMD:R_0402_1005Metric, symbol Device:R_Small
- removed R49: 120R, Resistor_SMD:R_0402_1005Metric, symbol Device:R_Small
- removed U4: MCP2515-xST, Package_SO:TSSOP-20_4.4x6.5mm_P0.65mm, symbol Interface_CAN_LIN:MCP2515-xST
- removed U5: TJA1051T-3, Package_SO:SOIC-8_3.9x4.9mm_P1.27mm, symbol Interface_CAN_LIN:TJA1051T-3
- removed Y3: 8MHz, Crystal:Crystal_SMD_Qantek_QC5CB-2Pin_5x3.2mm, symbol Device:Crystal_Small
- added C51: 22pF, Capacitor_SMD:C_0402_1005Metric, symbol Device:C_Small
- added R19: 10k, Resistor_SMD:R_0402_1005Metric, symbol Device:R_Small
- added R20: 120R, Resistor_SMD:R_0402_1005Metric, symbol Device:R_Small
- added SB5: SolderJumper_2_Open, Jumper:SolderJumper-2_P1.3mm_Open_TrianglePad1.0x1.5mm, symbol Jumper:SolderJumper_2_Open
- added U4: MCP25625, Package_DFN_QFN:QFN-28-1EP_6x6mm_P0.65mm_EP4.25x4.25mm, symbol Interface_CAN_LIN:MCP25625-x-SS
- added Y3: 16MHz, Crystal:Crystal_SMD_3225-4Pin_3.2x2.5mm, symbol Device:Crystal_GND2
- C47, C48: value 12pF -> 100nF; JLCPCB Part # (none) -> C1525; MFR.Part # (none) -> CL05B104KO5NNNC
- C50: value 100nF -> 22pF; JLCPCB Part # C1525 -> (none); MFR.Part # CL05B104KO5NNNC -> (none)
Connections:
- net +5V: now also C49.1, U4.27 (VDDA)
- net CAN_H: now also R20.1, U4.4 (CANH)
- net CAN_L: now also SB5.1 (A), U4.3 (CANL)
- net GND: now also C47.2, C51.1, U4.10 (GND), U4.26 (VSS), U4.5 (STBY), Y3.2; no longer C47.1
- net SPI_CLK: now also U4.14 (SCK)
- net SPI_MISO: now also U4.16 (SO)
- net SPI_MOSI: now also U4.15 (SI)
- net SPI_~{CS}: now also U4.17 (~{CS})
- net VCC: now also C47.1, C48.1, R19.1, U4.1 (VIO), U4.19 (VDD); no longer C49.1, C50.1
- net ~{INT}: now also U4.13 (~{INT})
- new net: C51.2, U4.9 (OSC1), Y3.1
- new net: C50.1, U4.8 (OSC2), Y3.3
- new net: R19.2, U4.18 (~{RESET})
- new net: U4.20 (TxCAN), U4.24 (TXD)
- new net: U4.21 (RxCAN), U4.28 (RXD)
- new net: R20.2, SB5.2 (B)
Other:
- note added: "The CLKOUT pin can provides the clock to the microcontroller."
- moved on the sheet: J8, J9

Commit message: Update ref
Parts:
- renumbered C47 to C44, C48 to C45, C49 to C46, C50 to C47, C51 to C48, J8 to J6, J9 to J7, R19 to R36, R20 to R37, SB5 to SB6, Y3 to Y2
Changed lines of the file:
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@@
   (symbol (lib_id "Device:Crystal_GND2") (at 144.78 121.92 90) (unit 1)
     (in_bom yes) (on_board yes) (fields_autoplaced)
-    (property "Reference" "Y3" (id 0) (at 140.97 120.6499 90)
+    (property "Reference" "Y2" (id 0) (at 140.97 120.6499 90)
       (effects (font (size 1.27 1.27)) (justify left))
     )
@@
   (symbol (lib_id "Device:C_Small") (at 132.08 73.66 90) (unit 1)
     (in_bom yes) (on_board yes)
-    (property "Reference" "C49" (id 0) (at 132.08 68.58 90))
+    (property "Reference" "C46" (id 0) (at 132.08 68.58 90))
     (property "Value" "100nF" (id 1) (at 132.08 71.12 90))
     (property "Footprint" "Capacitor_SMD:C_0402_1005Metric" (id 2) (at 132.08 73.66 0)
@@
   (symbol (lib_id "power:GND") (at 85.09 90.17 0) (mirror y) (unit 1)
     (in_bom yes) (on_board yes)
-    (property "Reference" "#PWR0115" (id 0) (at 85.09 96.52 0)
+    (property "Reference" "#PWR065" (id 0) (at 85.09 96.52 0)
       (effects (font (size 1.27 1.27)) hide)
     )
@@
   (symbol (lib_id "power:+5V") (at 124.46 73.66 0) (unit 1)
     (in_bom yes) (on_board yes)
-    (property "Reference" "#PWR0114" (id 0) (at 124.46 77.47 0)
+    (property "Reference" "#PWR069" (id 0) (at 124.46 77.47 0)
       (effects (font (size 1.27 1.27)) hide)
     )
@@
   (symbol (lib_id "power:VCC") (at 76.2 102.87 0) (mirror y) (unit 1)
     (in_bom yes) (on_board yes)
-    (property "Reference" "#PWR0112" (id 0) (at 76.2 106.68 0)
+    (property "Reference" "#PWR064" (id 0) (at 76.2 106.68 0)
       (effects (font (size 1.27 1.27)) hide)
     )
@@
   (symbol (lib_id "Device:C_Small") (at 106.68 73.66 270) (mirror x) (unit 1)
     (in_bom yes) (on_board yes)
-    (property "Reference" "C47" (id 0) (at 106.68 68.58 90))
+    (property "Reference" "C44" (id 0) (at 106.68 68.58 90))
     (property "Value" "100nF" (id 1) (at 106.68 71.12 90))
     (property "Footprint" "Capacitor_SMD:C_0402_1005Metric" (id 2) (at 106.68 73.66 0)
@@
   (symbol (lib_id "Device:C_Small") (at 151.13 118.11 90) (unit 1)
     (in_bom yes) (on_board yes)
-    (property "Reference" "C50" (id 0) (at 151.13 111.76 90))
+    (property "Reference" "C47" (id 0) (at 151.13 111.76 90))
     (property "Value" "22pF" (id 1) (at 151.13 114.3 90))
     (property "Footprint" "Capacitor_SMD:C_0402_1005Metric" (id 2) (at 151.13 118.11 0)
@@
   (symbol (lib_id "Device:R_Small") (at 76.2 105.41 0) (mirror y) (unit 1)
     (in_bom yes) (on_board yes)
-    (property "Reference" "R19" (id 0) (at 74.93 104.14 0)
+    (property "Reference" "R36" (id 0) (at 74.93 104.14 0)
       (effects (font (size 1.27 1.27)) (justify left))
     )
@@
   (symbol (lib_id "power:GND") (at 207.01 107.95 270) (unit 1)
     (in_bom yes) (on_board yes)
-    (property "Reference" "#PWR095" (id 0) (at 200.66 107.95 0)
+    (property "Reference" "#PWR074" (id 0) (at 200.66 107.95 0)
       (effects (font (size 1.27 1.27)) hide)
     )
@@
   (symbol (lib_id "power:GND") (at 207.01 93.98 270) (unit 1)
     (in_bom yes) (on_board yes)
-    (property "Reference" "#PWR094" (id 0) (at 200.66 93.98 0)
+    (property "Reference" "#PWR073" (id 0) (at 200.66 93.98 0)
       (effects (font (size 1.27 1.27)) hide)
     )
@@
   (symbol (lib_id "power:GND") (at 160.02 121.92 90) (unit 1)
     (in_bom yes) (on_board yes)
-    (property "Reference" "#PWR0109" (id 0) (at 166.37 121.92 0)
+    (property "Reference" "#PWR072" (id 0) (at 166.37 121.92 0)
       (effects (font (size 1.27 1.27)) hide)
     )
@@
   (symbol (lib_id "Device:R_Small") (at 177.8 95.25 0) (unit 1)
     (in_bom yes) (on_board yes)
-    (property "Reference" "R20" (id 0) (at 179.07 93.98 0)
+    (property "Reference" "R37" (id 0) (at 179.07 93.98 0)
       (effects (font (size 1.27 1.27)) (justify left))
     )
@@
   (symbol (lib_id "Device:C_Small") (at 106.68 78.74 270) (mirror x) (unit 1)
     (in_bom yes) (on_board yes)
-    (property "Reference" "C48" (id 0) (at 106.68 83.82 90))
+    (property "Reference" "C45" (id 0) (at 106.68 83.82 90))
     (property "Value" "100nF" (id 1) (at 106.68 81.28 90))
     (property "Footprint" "Capacitor_SMD:C_0402_1005Metric" (id 2) (at 106.68 78.74 0)
@@
   (symbol (lib_id "power:GND") (at 124.46 140.97 0) (unit 1)
     (in_bom yes) (on_board yes)
-    (property "Reference" "#PWR0116" (id 0) (at 124.46 147.32 0)
+    (property "Reference" "#PWR070" (id 0) (at 124.46 147.32 0)
       (effects (font (size 1.27 1.27)) hide)
     )
@@
   (symbol (lib_id "power:GND") (at 100.33 78.74 0) (mirror y) (unit 1)
     (in_bom yes) (on_board yes)
-    (property "Reference" "#PWR0111" (id 0) (at 100.33 85.09 0)
+    (property "Reference" "#PWR066" (id 0) (at 100.33 85.09 0)
       (effects (font (size 1.27 1.27)) hide)
     )
@@
   (symbol (lib_id "power:GND") (at 138.43 73.66 0) (unit 1)
     (in_bom yes) (on_board yes)
-    (property "Reference" "#PWR0113" (id 0) (at 138.43 80.01 0)
+    (property "Reference" "#PWR071" (id 0) (at 138.43 80.01 0)
       (effects (font (size 1.27 1.27)) hide)
     )
@@
   (symbol (lib_id "Connector_Generic:Conn_01x03") (at 218.44 93.98 0) (unit 1)
     (in_bom yes) (on_board yes)
-    (property "Reference" "J8" (id 0) (at 222.25 93.98 0))
+    (property "Reference" "J6" (id 0) (at 222.25 93.98 0))
     (property "Value" "Conn_02x02_Top_Bottom" (id 1) (at 219.71 100.33 0)
       (effects (font (size 1.27 1.27)) hide)
@@
   (symbol (lib_id "power:VCC") (at 114.3 73.66 0) (unit 1)
     (in_bom yes) (on_board yes)
-    (property "Reference" "#PWR0110" (id 0) (at 114.3 77.47 0)
+    (property "Reference" "#PWR067" (id 0) (at 114.3 77.47 0)
       (effects (font (size 1.27 1.27)) hide)
     )
@@
   (symbol (lib_id "power:GND") (at 116.84 140.97 0) (unit 1)
     (in_bom yes) (on_board yes)
-    (property "Reference" "#PWR0117" (id 0) (at 116.84 147.32 0)
+    (property "Reference" "#PWR068" (id 0) (at 116.84 147.32 0)
       (effects (font (size 1.27 1.27)) hide)
     )
@@
   (symbol (lib_id "Jumper:SolderJumper_2_Open") (at 177.8 101.6 90) (unit 1)
     (in_bom yes) (on_board yes) (fields_autoplaced)
-    (property "Reference" "SB5" (id 0) (at 180.34 101.5999 90)
+    (property "Reference" "SB6" (id 0) (at 180.34 101.5999 90)
       (effects (font (size 1.27 1.27)) (justify right))
     )
@@
   (symbol (lib_id "Connector_Generic:Conn_01x03") (at 218.44 107.95 0) (unit 1)
     (in_bom yes) (on_board yes)
-    (property "Reference" "J9" (id 0) (at 222.25 107.95 0))
+    (property "Reference" "J7" (id 0) (at 222.25 107.95 0))
     (property "Value" "Conn_02x02_Top_Bottom" (id 1) (at 219.71 114.3 0)
       (effects (font (size 1.27 1.27)) hide)
@@
   (symbol (lib_id "Device:C_Small") (at 151.13 125.73 270) (unit 1)
     (in_bom yes) (on_board yes)
-    (property "Reference" "C51" (id 0) (at 151.13 132.08 90))
+    (property "Reference" "C48" (id 0) (at 151.13 132.08 90))
     (property "Value" "22pF" (id 1) (at 151.13 129.54 90))
     (property "Footprint" "Capacitor_SMD:C_0402_1005Metric" (id 2) (at 151.13 125.73 0)

Commit message: Use kelvin connection for shunt resistance
Parts:
- C47, C48: JLCPCB Part # (none) -> C1653; MFR.Part # (none) -> CL10C220JB8NNNC
- J6, J7: JLCPCB Part # (none) -> C2829252; MFR.Part # (none) -> GH1.25-3PWBPZ
- SB6: now left out of the parts list
Changed lines of the file:
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@@
+      (effects (font (size 1.27 1.27)) hide)
+    )
+    (property "JLCPCB Part #" "C1653" (id 4) (at 151.13 118.11 0)
+      (effects (font (size 1.27 1.27)) hide)
+    )
+    (property "MFR.Part #" "CL10C220JB8NNNC" (id 5) (at 151.13 118.11 0)
       (effects (font (size 1.27 1.27)) hide)
     )
@@
       (effects (font (size 1.27 1.27)) hide)
     )
-    (property "JLCPCB Part #" "" (id 4) (at 218.44 93.98 0)
-      (effects (font (size 1.27 1.27)) hide)
-    )
-    (property "MFR.Part #" "" (id 5) (at 218.44 93.98 0)
+    (property "JLCPCB Part #" "C2829252" (id 4) (at 218.44 93.98 0)
+      (effects (font (size 1.27 1.27)) hide)
+    )
+    (property "MFR.Part #" "GH1.25-3PWBPZ" (id 5) (at 218.44 93.98 0)
       (effects (font (size 1.27 1.27)) hide)
     )
@@
   )
   (symbol (lib_id "Jumper:SolderJumper_2_Open") (at 177.8 101.6 90) (unit 1)
-    (in_bom yes) (on_board yes) (fields_autoplaced)
+    (in_bom no) (on_board yes) (fields_autoplaced)
     (property "Reference" "SB6" (id 0) (at 180.34 101.5999 90)
       (effects (font (size 1.27 1.27)) (justify right))
@@
       (effects (font (size 1.27 1.27)) hide)
     )
-    (property "JLCPCB Part #" "" (id 4) (at 218.44 107.95 0)
-      (effects (font (size 1.27 1.27)) hide)
-    )
-    (property "MFR.Part #" "" (id 5) (at 218.44 107.95 0)
+    (property "JLCPCB Part #" "C2829252" (id 4) (at 218.44 107.95 0)
+      (effects (font (size 1.27 1.27)) hide)
+    )
+    (property "MFR.Part #" "GH1.25-3PWBPZ" (id 5) (at 218.44 107.95 0)
       (effects (font (size 1.27 1.27)) hide)
     )
@@
       (effects (font (size 1.27 1.27)) hide)
     )
+    (property "JLCPCB Part #" "C1653" (id 4) (at 151.13 125.73 0)
+      (effects (font (size 1.27 1.27)) hide)
+    )
+    (property "MFR.Part #" "CL10C220JB8NNNC" (id 5) (at 151.13 125.73 0)
+      (effects (font (size 1.27 1.27)) hide)
+    )

Commit message: Replace some extended parts to basic parts
Parts:
- C44, C45, C46, C47, C48, R36, R37: Basic Part (none) -> Y
- J6, J7, U4: Basic Part (none) -> N
- Y2: Basic Part (none) -> Y; JLCPCB Part # C156247 -> C13738; MFR.Part # NX3225GA-16MHZ-STD-CRG-2 -> X322516MLB4SI
Changed lines of the file:
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@@
       (effects (font (size 1.27 1.27)) hide)
     )
-    (property "JLCPCB Part #" "C156247" (id 4) (at 144.78 121.92 0)
-      (effects (font (size 1.27 1.27)) hide)
-    )
-    (property "MFR.Part #" "NX3225GA-16MHZ-STD-CRG-2" (id 5) (at 144.78 121.92 0)
+    (property "JLCPCB Part #" "C13738" (id 4) (at 144.78 121.92 0)
+      (effects (font (size 1.27 1.27)) hide)
+    )
+    (property "MFR.Part #" "X322516MLB4SI" (id 5) (at 144.78 121.92 0)
+      (effects (font (size 1.27 1.27)) hide)
+    )
+    (property "Basic Part" "Y" (id 6) (at 144.78 121.92 0)
       (effects (font (size 1.27 1.27)) hide)
     )
@@
       (effects (font (size 1.27 1.27)) hide)
     )
+    (property "Basic Part" "Y" (id 6) (at 132.08 73.66 0)
+      (effects (font (size 1.27 1.27)) hide)
+    )
     (pin "1")
     (pin "2")
@@
       (effects (font (size 1.27 1.27)) hide)
     )
+    (property "Basic Part" "Y" (id 6) (at 106.68 73.66 0)
+      (effects (font (size 1.27 1.27)) hide)
+    )
     (pin "1")
     (pin "2")
@@
       (effects (font (size 1.27 1.27)) hide)
     )
+    (property "Basic Part" "Y" (id 6) (at 151.13 118.11 0)
+      (effects (font (size 1.27 1.27)) hide)
+    )
     (pin "1")
     (pin "2")
@@
     )
     (property "MFR.Part #" "0402WGF1002TCE" (id 5) (at 76.2 105.41 0)
+      (effects (font (size 1.27 1.27)) hide)
+    )
+    (property "Basic Part" "Y" (id 6) (at 76.2 105.41 0)
       (effects (font (size 1.27 1.27)) hide)
     )
@@
     )
     (property "MFR.Part #" "MCP25625T-E/ML" (id 5) (at 119.38 113.03 0)
+      (effects (font (size 1.27 1.27)) hide)
+    )
+    (property "Basic Part" "N" (id 6) (at 119.38 113.03 0)
       (effects (font (size 1.27 1.27)) hide)
     )
@@
       (effects (font (size 1.27 1.27)) hide)
     )
+    (property "Basic Part" "Y" (id 6) (at 177.8 95.25 0)
+      (effects (font (size 1.27 1.27)) hide)
+    )
     (pin "1")
     (pin "2")
@@
       (effects (font (size 1.27 1.27)) hide)
     )
+    (property "Basic Part" "Y" (id 6) (at 106.68 78.74 0)
+      (effects (font (size 1.27 1.27)) hide)
+    )
     (pin "1")
     (pin "2")
@@
     )
     (property "MFR.Part #" "GH1.25-3PWBPZ" (id 5) (at 218.44 93.98 0)
+      (effects (font (size 1.27 1.27)) hide)
+    )
+    (property "Basic Part" "N" (id 6) (at 218.44 93.98 0)
       (effects (font (size 1.27 1.27)) hide)
     )
@@
       (effects (font (size 1.27 1.27)) hide)
     )
+    (property "Basic Part" "" (id 4) (at 177.8 101.6 0)
+      (effects (font (size 1.27 1.27)) hide)
+    )
     (pin "1")
     (pin "2")
@@
     )
     (property "MFR.Part #" "GH1.25-3PWBPZ" (id 5) (at 218.44 107.95 0)
+      (effects (font (size 1.27 1.27)) hide)
+    )
+    (property "Basic Part" "N" (id 6) (at 218.44 107.95 0)
       (effects (font (size 1.27 1.27)) hide)
     )
@@
       (effects (font (size 1.27 1.27)) hide)
     )
+    (property "Basic Part" "Y" (id 6) (at 151.13 125.73 0)
+      (effects (font (size 1.27 1.27)) hide)
+    )

Commit message: Update C47, C48 to the correct part number
Parts:
- C47, C48: JLCPCB Part # C1653 -> C1555; MFR.Part # CL10C220JB8NNNC -> 0402CG220J500NT
Changed lines of the file:
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@@
       (effects (font (size 1.27 1.27)) hide)
     )
-    (property "JLCPCB Part #" "C1653" (id 4) (at 151.13 118.11 0)
-      (effects (font (size 1.27 1.27)) hide)
-    )
-    (property "MFR.Part #" "CL10C220JB8NNNC" (id 5) (at 151.13 118.11 0)
+    (property "JLCPCB Part #" "C1555" (id 4) (at 151.13 118.11 0)
+      (effects (font (size 1.27 1.27)) hide)
+    )
+    (property "MFR.Part #" "0402CG220J500NT" (id 5) (at 151.13 118.11 0)
       (effects (font (size 1.27 1.27)) hide)
     )
@@
       (effects (font (size 1.27 1.27)) hide)
     )
-    (property "JLCPCB Part #" "C1653" (id 4) (at 151.13 125.73 0)
-      (effects (font (size 1.27 1.27)) hide)
-    )
-    (property "MFR.Part #" "CL10C220JB8NNNC" (id 5) (at 151.13 125.73 0)
-      (effects (font (size 1.27 1.27)) hide)
-    )
+    (property "JLCPCB Part #" "C1555" (id 4) (at 151.13 125.73 0)
+      (effects (font (size 1.27 1.27)) hide)
+    )
+    (property "MFR.Part #" "0402CG220J500NT" (id 5) (at 151.13 125.73 0)
+      (effects (font (size 1.27 1.27)) hide)
+    )
