File: hardware/moco-o/moco-o.kicad_sch (KiCad schematic)
At the start: 93 parts, among them J1 USB_C_Receptacle_USB2.0, J2 Conn_02x10_Odd_Even, J3 Conn_01x02, J4 Conn_01x05, J5 SWD 10-Pin, J6 ST-LINK, J8 Conn_01x06, J9 Conn_01x06, Q1 AO3413, Q2 AO3413, SW1 SW_Push, SW2 SW_Push, SW3 SW_Push, SW4 SW_Push, U1 AMS1117-3.3

Commit message: Change to DRV8323H
Parts:
- removed C3, C4, C5, C7: 82pF, Capacitor_SMD:C_0402_1005Metric, symbol Device:C_Small
- removed C6: 270pF, Capacitor_SMD:C_0402_1005Metric, symbol Device:C
- removed C8: 10uF, Capacitor_SMD:C_0402_1005Metric, symbol Device:C
- removed C9: 10uF, Capacitor_Tantalum_SMD:CP_EIA-3216-18_Kemet-A, symbol Device:C_Polarized
- removed D1: SS34, Diode_SMD:D_SMA, symbol Diode:MBR340
- removed F1: 500mA/6V, Fuse:Fuse_0805_2012Metric, symbol Device:Polyfuse
- removed H1, H2: MountingHole_Pad, MountingHole:MountingHole_3.2mm_M3_Pad_Via, symbol Mechanical:MountingHole_Pad
- removed H3: MountingHole, MountingHole:MountingHole_3.2mm_M3_ISO14580, symbol Mechanical:MountingHole
- removed J1: USB_C_Receptacle_USB2.0, Connector_USB:USB_C_Receptacle_HRO_TYPE-C-31-M-12, symbol Connector:USB_C_Receptacle_USB2.0
- removed J2: Conn_02x10_Odd_Even, Connector_PinHeader_2.54mm:PinHeader_2x08_P2.54mm_Vertical, symbol Connector_Generic:Conn_02x08_Odd_Even
- removed J3: Conn_01x02, Connector_AMASS:AMASS_XT60-M_1x02_P7.20mm_Vertical, symbol Connector_Generic:Conn_01x02
- removed J4: Conn_01x05, Connector_JST:JST_GH_SM05B-GHS-TB_1x05-1MP_P1.25mm_Horizontal, symbol Connector_Generic:Conn_01x05
- removed J5: SWD 10-Pin, Connector_PinHeader_1.27mm:PinHeader_2x05_P1.27mm_Vertical_SMD, symbol Connector_Generic:Conn_02x05_Odd_Even
- removed J6: ST-LINK, Connector_PinHeader_2.54mm:PinHeader_1x05_P2.54mm_Vertical, symbol Connector_Generic:Conn_01x05
- removed J8: Conn_01x06, Connector_JST:JST_GH_SM06B-GHS-TB_1x06-1MP_P1.25mm_Horizontal, symbol Connector_Generic:Conn_01x06
- removed J9: Conn_01x06, Connector_JST:JST_GH_BM06B-GHS-TBT_1x06-1MP_P1.25mm_Vertical, symbol Connector_Generic:Conn_01x06
- removed JP1: Jumper_3_Open, Connector_PinHeader_2.54mm:PinHeader_1x03_P2.54mm_Vertical_SMD_Pin1Left, symbol Jumper:Jumper_3_Open
- removed LD1, LD2, LD3, LD4, LD5, LD6: LED, LED_SMD:LED_0603_1608Metric, symbol Device:LED
- removed Q1, Q2: AO3413, Package_TO_SOT_SMD:SOT-23, symbol Transistor_FET:AO3401A
- removed R1, R10, R2, R20, R23, R3, R9: 10k, Resistor_SMD:R_0402_1005Metric, symbol Device:R
- removed R11, R12: 5.1k, Resistor_SMD:R_0402_1005Metric, symbol Device:R
- removed R13, R24, R29: 1k, Resistor_SMD:R_0402_1005Metric, symbol Device:R
- removed R14, R19, R21, R22, R25: 3.3k, Resistor_SMD:R_0402_1005Metric, symbol Device:R_Small
- removed R15, R16: 330R, Resistor_SMD:R_0402_1005Metric, symbol Device:R
- removed R17, R18: 22R, Resistor_SMD:R_0402_1005Metric, symbol Device:R
- removed R26, R27, R28: 3.3k, Resistor_SMD:R_0402_1005Metric, symbol Device:R
- removed R7, R8: 150R, Resistor_SMD:R_0402_1005Metric, symbol Device:R
- removed SB1, SB11, SB13, SB15, SB17, SB19, SB2, SB20, SB22, SB3, SB4, SB5, SB6, SB7, SB9: SolderJumper_2_Bridged, Jumper:SolderJumper-2_P1.3mm_Bridged_RoundedPad1.0x1.5mm, symbol Jumper:SolderJumper_2_Bridged
- removed SB10, SB12, SB14, SB16, SB8: SolderJumper_2_Open, Jumper:SolderJumper-2_P1.3mm_Open_RoundedPad1.0x1.5mm, symbol Jumper:SolderJumper_2_Open
- removed SB18, SB21: SolderJumper_3_Bridged12, Jumper:SolderJumper-3_P1.3mm_Bridged12_RoundedPad1.0x1.5mm_NumberLabels, symbol Jumper:SolderJumper_3_Bridged12
- removed SW1, SW2, SW3, SW4: SW_Push, Button_Switch_SMD:SW_SPST_CK_RS282G05A3, symbol Switch:SW_Push
- removed TH1: NCP18XH103F03RB, Resistor_SMD:R_0603_1608Metric, symbol Device:Thermistor_NTC
- removed TP1, TP2: TestPoint_Small, TestPoint:TestPoint_Pad_D2.0mm, symbol Connector:TestPoint_Small
- removed TP3, TP4: TestPoint, TestPoint:TestPoint_Pad_D2.0mm, symbol Connector:TestPoint
- removed U1: AMS1117-3.3, Package_TO_SOT_SMD:SOT-223-3_TabPin2, symbol Regulator_Linear:AMS1117-3.3
- added C3: 10uF, Capacitor_SMD:C_0603_1608Metric, symbol Device:C
- added C4, C5: 1uF, Capacitor_SMD:C_0402_1005Metric, symbol Device:C
- added D?: SS34, Diode_SMD:D_SMA, symbol Diode:MBR340
- added H1, H2: MountingHole, MountingHole:MountingHole_3.2mm_M3_ISO14580, symbol Mechanical:MountingHole
- added J1: Serial, Connector_JST:JST_GH_BM03B-GHS-TBT_1x03-1MP_P1.25mm_Vertical, symbol Connector_Generic:Conn_01x03
- added J2: Debug, Connector_PinHeader_2.54mm:PinHeader_2x04_P2.54mm_Vertical, symbol Connector_Generic:Conn_02x04_Odd_Even
- added J? (x2): A, moco:wire_3.2mm, symbol Connector_Generic:Conn_01x01
- added L1: 22uH, Inductor_SMD:L_7.3x7.3_H3.5, symbol Device:L
- added LD1: LED_BAGR, moco:RGB LED 1.6x1.6mm, symbol Device:LED_BAGR
- added R1: 54.9k, Resistor_SMD:R_0402_1005Metric, symbol Device:R_Small
- added R3: 10k, Resistor_SMD:R_0402_1005Metric, symbol Device:R_Small
- added R?: 10k, Resistor_SMD:R_0402_1005Metric, symbol Device:R
- added TH?: NCP18XH103F03RB, Resistor_SMD:R_0603_1608Metric, symbol Device:Thermistor_NTC
- added U1: LMR16006X, Package_TO_SOT_SMD:SOT-23-6, symbol Regulator_Switching:LMR16006YQ
- added U2: RT9013-33GB, Package_TO_SOT_SMD:SOT-23-5, symbol Regulator_Linear:XC6220B331MR
- C1: value 82pF -> 100nF; JLCPCB Part # C107011 -> (none); MFR.Part # CC0402JRNPO9BN820 -> (none)
- C2: value 2.2uF -> 1uF/50V; footprint Capacitor_SMD:C_0402_1005Metric -> Capacitor_SMD:C_1206_3216Metric; JLCPCB Part # C501836 -> (none); MFR.Part # 0402X225K160NT -> (none)
- R4: value 10k -> 1k; JLCPCB Part # C25744 -> C25130; MFR.Part # 0402WGF1002TCE -> 0402WGF6800TCE
- R5: value 1k -> 5k
- R6: JLCPCB Part # C11702 -> C25104; MFR.Part # 0402WGF1001TCE -> 0402WGF3300TCE
- renumbered H4 to H3
Connections:
- net MCU_~{RESET} is gone; now on net USER_LED1: R4.2
- net POWER_TEMP is gone; now on net Vdrive: C2.1
- net +5V: now also C3.1, C4.1, J2.2 (Pin_2), L1.2, LD1.2 (A), R1.1, U2.1 (VIN), U2.3 (CE)
- net GND: now also R5.2, C3.2, C4.2, C5.2, D?.2 (A), J1.3 (Pin_3), J2.7 (Pin_7), J2.8 (Pin_8), R3.2, R?.1, U1.2 (GND), U2.2 (GND); no longer C1.2
- net SWCLK: now also J2.4 (Pin_4)
- net SWDIO: now also J2.6 (Pin_6)
- net USER_LED2: now also R6.2
- net Vdrive: now also J?.1 (Pin_1), U1.5 (VIN)
- net at R5.1: now also LD1.3 (GK)
- net at R6.1: now also LD1.1 (BK)
- net at C1.1: now also U1.1 (CB)
- net VCC: no longer names the net of R4.1
- net VCC: now also LD1.4 (RK)
- new net: R1.2, R3.1, U1.3 (FB)
- new net: C1.2, D?.1 (K), L1.1, U1.6 (SW)
- new net +3.3V: C5.1, J2.1 (Pin_1), TH?.1, U2.5 (VOUT)
- new net GNDPWR: J?.1 (Pin_1)
- new net TEMP_SENSOR: R?.2, TH?.2
- new net UART1_RX: J2.5 (Pin_5)
- new net UART1_TX: J2.3 (Pin_3)
- new net UART2_RX: J1.2 (Pin_2)
- new net UART2_TX: J1.1 (Pin_1)
- no-connect marks 6 -> 4
Other:
- sheet Rotary Position Sensor renamed Angle Sensor
- removed sheet Braking Circuit
- removed sheet CAN BUS
- added sheet CAN Bus (can_bus.kicad_sch)
- sheet Angle Sensor ports: added MISO, MOSI, SCLK, ~{CS}; removed SPI_CLK, SPI_MISO, SPI_MOSI, SPI_~{CS}
- sheet MCU ports: added AMP_CAL, CAN_RX, CAN_TX, CS_A, CS_B, CS_C, GATE_ENABLE, PWM_HA, PWM_HB, PWM_HC, PWM_LA, PWM_LB, PWM_LC, SPI1_MISO, SPI1_MOSI, SPI1_SCK, SPI1_~{CS}_AS5047, TEMP, UART1_RX, UART1_TX, UART2_RX, UART2_TX, VREF; removed AUX_H, AUX_L, AUX_TEMP, CAN_BUS_RX, CAN_BUS_TX, EN_GATE, GPIO_PA0, GPIO_PA1, GPIO_PA15, GPIO_PA2, GPIO_PA3, GPIO_PA7, GPIO_PB0, GPIO_PB1, GPIO_PB2, GPIO_PB3, GPIO_PC4, GPIO_PC8, M0_AH, M0_AL, M0_BH, M0_BL, M0_CH, M0_CL, M0_CUR_SENSE_1, M0_CUR_SENSE_2, M0_ENC_A, M0_ENC_B, M0_ENC_Z, M0_TEMP, POWER_TEMP, SENSOR_ENC_A, SENSOR_ENC_B, SENSOR_ENC_Z, SPI_CLK, SPI_MISO, SPI_MOSI, SPI_~{CS}_M0, SPI_~{CS}_SENSOR, USB_D+, USB_D-, USER_Button1, USER_Button2, VBUS_S
- sheet Motor Driver ports: added CAL, ENABLE, INHA, INHB, INHC, INLA, INLB, INLC, SOA, SOB, SOC, VREF; removed CUR_SENSE_1, CUR_SENSE_2, EN_GATE, INH_A, INH_B, INH_C, INL_A, INL_B, INL_C, PWRGD, SPI_CLK, SPI_MISO, SPI_MOSI, SPI_~{CS}, TEMP_SENSE, ~{OCTW}
- note added: "LED Forward Voltage (V_{F}): R: 1.9~2.2V G: 2.9~3.4V B: 2.9~3.4V"
- note removed: "+5V from DRV8301 integrated buck converter"
- note removed: "SWO"
- title: MoCo-O -> moco-OD501
