File: hardware/moco8316/moco8316.kicad_pcb (KiCad board)
At the start: 2 copper layers, 55 parts, among them J1 Conn_01x02, J2 Conn_02x10_Odd_Even, J3 Conn_01x03, U1 RT9013-33GB, U2 DRV8316CR, U3 LM4040D33FTA

Commit message: Update edge
Parts:
- added J4: Conn_01x01, moco:wire_3.2mm, F.Cu at (161.0, 117.0)
- added J5: Conn_01x01, moco:wire_3.2mm, F.Cu at (161.0, 103.0)
- J3: value Conn_01x03 -> Conn_01x01; footprint Connector_Wire:SolderWire-2.5sqmm_1x03_P7.2mm_D2.4mm_OD3.6mm -> moco:wire_3.2mm
- moved H4 60.6 mm to (119.0, 91.5)
- moved H2 53.6 mm to (161.0, 91.5)
- moved H1 43.4 mm to (119.0, 128.5)
- moved J2 15.2 mm to (119.3, 98.6)
- moved J3 14.3 mm to (161.0, 110.0), turned to 0 degrees
- moved H3 10.4 mm to (161.0, 128.5)
- moved C1 10.3 mm to (146.2, 116.0)
- moved C10 10.3 mm to (132.8, 115.8)
- moved C11 10.3 mm to (139.8, 113.5)
- moved C12 10.3 mm to (136.2, 113.5)
- moved C13 10.3 mm to (132.8, 113.5)
- moved C15 10.3 mm to (155.5, 119.8)
- moved C16 10.3 mm to (153.2, 119.8)
- moved C17 10.3 mm to (151.0, 119.8)
- moved C18 10.3 mm to (148.8, 119.8)
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Connections:
- J3 pad 1: /OUT_A -> /OUT_B
Other:
- board outline added: 50 x 45 mm
