File: hardware/moco8316/moco8316.kicad_sch (KiCad schematic)
At the start: 55 parts, among them J1 Conn_01x02, J2 Conn_02x10_Odd_Even, J3 Conn_01x03, U1 RT9013-33GB, U2 DRV8316CR, U3 LM4040D33FTA

Commit message: Update edge
Parts:
- removed J3: Conn_01x03, Connector_Wire:SolderWire-2.5sqmm_1x03_P7.2mm_D2.4mm_OD3.6mm, symbol Connector_Generic:Conn_01x03
- added J3, J4, J5: Conn_01x01, moco:wire_3.2mm, symbol Connector_Generic:Conn_01x01
Connections:
- net OUT_A: now also J4.1 (Pin_1)
- net OUT_B: now also J3.1 (Pin_1)
- net OUT_C: now also J5.1 (Pin_1)
Changed lines of the file:
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@@
+    )
+  )
+  (symbol (lib_id "Connector_Generic:Conn_01x01") (at 179.07 118.11 0) (unit 1)
+    (in_bom yes) (on_board yes) (dnp no)
+    (property "Reference" "J4" (at 181.61 118.11 0)
+      (effects (font (size 1.27 1.27)) (justify left))
+    )
+    (property "Value" "Conn_01x01" (at 181.61 119.38 0)
+      (effects (font (size 1.27 1.27)) (justify left) hide)
+    )
+    (property "Footprint" "moco:wire_3.2mm" (at 179.07 118.11 0)
+      (effects (font (size 1.27 1.27)) hide)
+    )
+    (property "Datasheet" "~" (at 179.07 118.11 0)
+      (effects (font (size 1.27 1.27)) hide)
+    )
+    (pin "1")
+    (instances
+      (project "moco8316"
+        (path "/60ff2a18-57fe-4fe9-a422-66a2356bfaaa"
+          (reference "J4") (unit 1)
+        )
+      )
     )
   )
@@
         (path "/60ff2a18-57fe-4fe9-a422-66a2356bfaaa"
           (reference "C20") (unit 1)
-        )
-      )
-    )
-  )
-  (symbol (lib_id "Connector_Generic:Conn_01x03") (at 179.07 120.65 0) (unit 1)
-    (in_bom yes) (on_board yes) (dnp no) (fields_autoplaced)
-    (property "Reference" "J3" (at 181.61 119.3799 0)
-      (effects (font (size 1.27 1.27)) (justify left))
-    )
-    (property "Value" "Conn_01x03" (at 181.61 121.9199 0)
-      (effects (font (size 1.27 1.27)) (justify left))
-    )
-    (property "Footprint" "Connector_Wire:SolderWire-2.5sqmm_1x03_P7.2mm_D2.4mm_OD3.6mm" (at 179.07 120.65 0)
-      (effects (font (size 1.27 1.27)) hide)
-    )
-    (property "Datasheet" "~" (at 179.07 120.65 0)
-      (effects (font (size 1.27 1.27)) hide)
-    )
-    (pin "1")
-    (pin "2")
-    (pin "3")
-    (instances
-      (project "moco8316"
-        (path "/60ff2a18-57fe-4fe9-a422-66a2356bfaaa"
-          (reference "J3") (unit 1)
         )
       )
@@
         (path "/60ff2a18-57fe-4fe9-a422-66a2356bfaaa"
           (reference "R10") (unit 1)
+        )
+      )
+    )
+  )
+  (symbol (lib_id "Connector_Generic:Conn_01x01") (at 179.07 123.19 0) (unit 1)
+    (in_bom yes) (on_board yes) (dnp no)
+    (property "Reference" "J5" (at 181.61 123.19 0)
+      (effects (font (size 1.27 1.27)) (justify left))
+    )
+    (property "Value" "Conn_01x01" (at 181.61 124.46 0)
+      (effects (font (size 1.27 1.27)) (justify left) hide)
+    )
+    (property "Footprint" "moco:wire_3.2mm" (at 179.07 123.19 0)
+      (effects (font (size 1.27 1.27)) hide)
+    )
+    (property "Datasheet" "~" (at 179.07 123.19 0)
+      (effects (font (size 1.27 1.27)) hide)
+    )
+    (pin "1")
+    (instances
+      (project "moco8316"
+        (path "/60ff2a18-57fe-4fe9-a422-66a2356bfaaa"
+          (reference "J5") (unit 1)
         )
       )
@@
         )
       )
+    )
+  )
+  (symbol (lib_id "Connector_Generic:Conn_01x01") (at 179.07 120.65 0) (unit 1)
+    (in_bom yes) (on_board yes) (dnp no)
+    (property "Reference" "J3" (at 181.61 120.65 0)
+      (effects (font (size 1.27 1.27)) (justify left))
+    )
+    (property "Value" "Conn_01x01" (at 181.61 121.92 0)
+      (effects (font (size 1.27 1.27)) (justify left) hide)
+    )
+    (property "Footprint" "moco:wire_3.2mm" (at 179.07 120.65 0)
+      (effects (font (size 1.27 1.27)) hide)
+    )
+    (property "Datasheet" "~" (at 179.07 120.65 0)
+      (effects (font (size 1.27 1.27)) hide)
+    )
+    (pin "1")
+    (instances
+      (project "moco8316"
+        (path "/60ff2a18-57fe-4fe9-a422-66a2356bfaaa"
+          (reference "J3") (unit 1)
+        )
+      )
