File: hardware/moco-oi401/mcu.kicad_sch (KiCad schematic)
At the start: 14 parts, among them SW1 RESET, U2 STM32G431CBUx, Y1 8MHz

Commit message: Update part#
Parts:
- C10, C3, C4, C5, C6, C9: JLCPCB Part # C1525 -> (none); LCSC (none) -> C1525; MFR. Part# (none) -> CL05B104KO5NNNC; MFR.Part # CL05B104KO5NNNC -> (none)
- C11, C12: LCSC (none) -> C1547; MFR. Part# (none) -> 0402CG120J500NT
- C7: JLCPCB Part # C1525 -> (none); LCSC (none) -> C15195; MFR. Part# (none) -> CL05B103KB5NNNC; MFR.Part # CL05B104KO5NNNC -> (none)
- C8: LCSC (none) -> C52923; MFR. Part# (none) -> CL05A105KA5NQNC
- SW1: LCSC (none) -> C5117871; MFR. Part# (none) -> GT-TC060B-H027-L1
- U2: JLCPCB Part # C529356 -> (none); LCSC (none) -> C529356; MFR. Part# (none) -> STM32G431CBU6; MFR.Part # STM32G431CBU6 -> (none)
- Y1: value 8MHz -> 16MHz; LCSC (none) -> C13738; MFR. Part# (none) -> X322516MLB4SI
Changed lines of the file:
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@@
       (effects (font (size 1.27 1.27)) hide)
     )
-    (property "JLCPCB Part #" "C1525" (at 123.19 64.77 0)
-      (effects (font (size 1.27 1.27)) hide)
-    )
-    (property "MFR.Part #" "CL05B104KO5NNNC" (at 123.19 64.77 0)
+    (property "LCSC" "C1525" (at 123.19 64.77 0)
+      (effects (font (size 1.27 1.27)) hide)
+    )
+    (property "MFR. Part#" "CL05B104KO5NNNC" (at 123.19 64.77 0)
       (effects (font (size 1.27 1.27)) hide)
     )
@@
       (effects (font (size 1.27 1.27)) hide)
     )
-    (property "JLCPCB Part #" "C1525" (at 175.26 41.91 0)
-      (effects (font (size 1.27 1.27)) hide)
-    )
-    (property "MFR.Part #" "CL05B104KO5NNNC" (at 175.26 41.91 0)
+    (property "LCSC" "C15195" (at 175.26 41.91 0)
+      (effects (font (size 1.27 1.27)) hide)
+    )
+    (property "MFR. Part#" "CL05B103KB5NNNC" (at 175.26 41.91 0)
       (effects (font (size 1.27 1.27)) hide)
     )
@@
       (effects (font (size 1.27 1.27)) hide)
     )
-    (property "JLCPCB Part #" "C1525" (at 138.43 41.91 0)
-      (effects (font (size 1.27 1.27)) hide)
-    )
-    (property "MFR.Part #" "CL05B104KO5NNNC" (at 138.43 41.91 0)
+    (property "LCSC" "C1525" (at 138.43 41.91 0)
+      (effects (font (size 1.27 1.27)) hide)
+    )
+    (property "MFR. Part#" "CL05B104KO5NNNC" (at 138.43 41.91 0)
       (effects (font (size 1.27 1.27)) hide)
     )
@@
       (effects (font (size 1.27 1.27)) hide)
     )
-    (property "JLCPCB Part #" "C1525" (at 64.77 76.2 0)
-      (effects (font (size 1.27 1.27)) hide)
-    )
-    (property "MFR.Part #" "CL05B104KO5NNNC" (at 64.77 76.2 0)
+    (property "LCSC" "C1525" (at 64.77 76.2 0)
+      (effects (font (size 1.27 1.27)) hide)
+    )
+    (property "MFR. Part#" "CL05B104KO5NNNC" (at 64.77 76.2 0)
       (effects (font (size 1.27 1.27)) hide)
     )
@@
       (effects (font (size 1.27 1.27)) hide)
     )
+    (property "LCSC" "C1547" (at 49.53 113.03 0)
+      (effects (font (size 1.27 1.27)) hide)
+    )
+    (property "MFR. Part#" "0402CG120J500NT" (at 49.53 113.03 0)
+      (effects (font (size 1.27 1.27)) hide)
+    )
     (pin "1")
     (pin "2")
@@
       (effects (font (size 1.27 1.27)) hide)
     )
+    (property "LCSC" "C1547" (at 49.53 120.65 0)
+      (effects (font (size 1.27 1.27)) hide)
+    )
+    (property "MFR. Part#" "0402CG120J500NT" (at 49.53 120.65 0)
+      (effects (font (size 1.27 1.27)) hide)
+    )
     (pin "1")
     (pin "2")
@@
       (effects (font (size 1.27 1.27)) hide)
     )
-    (property "JLCPCB Part #" "C1525" (at 130.81 41.91 0)
-      (effects (font (size 1.27 1.27)) hide)
-    )
-    (property "MFR.Part #" "CL05B104KO5NNNC" (at 130.81 41.91 0)
+    (property "LCSC" "C1525" (at 130.81 41.91 0)
+      (effects (font (size 1.27 1.27)) hide)
+    )
+    (property "MFR. Part#" "CL05B104KO5NNNC" (at 130.81 41.91 0)
       (effects (font (size 1.27 1.27)) hide)
     )
@@
       (effects (font (size 1.27 1.27)) hide)
     )
+    (property "LCSC" "C5117871" (at 59.69 76.2 0)
+      (effects (font (size 1.27 1.27)) hide)
+    )
+    (property "MFR. Part#" "GT-TC060B-H027-L1" (at 59.69 76.2 0)
+      (effects (font (size 1.27 1.27)) hide)
+    )
     (pin "1")
     (pin "2")
@@
       (effects (font (size 1.27 1.27)))
     )
-    (property "Value" "8MHz" (at 58.42 123.19 90)
+    (property "Value" "16MHz" (at 58.42 123.19 90)
       (effects (font (size 1.27 1.27)))
     )
@@
     )
     (property "Datasheet" "~" (at 58.42 116.84 0)
+      (effects (font (size 1.27 1.27)) hide)
+    )
+    (property "LCSC" "C13738" (at 58.42 116.84 0)
+      (effects (font (size 1.27 1.27)) hide)
+    )
+    (property "MFR. Part#" "X322516MLB4SI" (at 58.42 116.84 0)
       (effects (font (size 1.27 1.27)) hide)
     )
@@
       (effects (font (size 1.27 1.27)) hide)
     )
-    (property "JLCPCB Part #" "C1525" (at 123.19 41.91 0)
-      (effects (font (size 1.27 1.27)) hide)
-    )
-    (property "MFR.Part #" "CL05B104KO5NNNC" (at 123.19 41.91 0)
+    (property "LCSC" "C1525" (at 123.19 41.91 0)
+      (effects (font (size 1.27 1.27)) hide)
+    )
+    (property "MFR. Part#" "CL05B104KO5NNNC" (at 123.19 41.91 0)
       (effects (font (size 1.27 1.27)) hide)
     )
@@
       (effects (font (size 1.27 1.27)) hide)
     )
+    (property "LCSC" "C52923" (at 182.88 41.91 0)
+      (effects (font (size 1.27 1.27)) hide)
+    )
+    (property "MFR. Part#" "CL05A105KA5NQNC" (at 182.88 41.91 0)
+      (effects (font (size 1.27 1.27)) hide)
+    )
     (pin "1")
     (pin "2")
@@
       (effects (font (size 1.27 1.27)) hide)
     )
-    (property "JLCPCB Part #" "C529356" (at 156.21 101.6 0)
-      (effects (font (size 1.27 1.27)) hide)
-    )
-    (property "MFR.Part #" "STM32G431CBU6" (at 156.21 101.6 0)
+    (property "LCSC" "C529356" (at 156.21 101.6 0)
+      (effects (font (size 1.27 1.27)) hide)
+    )
+    (property "MFR. Part#" "STM32G431CBU6" (at 156.21 101.6 0)
       (effects (font (size 1.27 1.27)) hide)
     )
@@
       (effects (font (size 1.27 1.27)) hide)
     )
-    (property "JLCPCB Part #" "C1525" (at 146.05 41.91 0)
-      (effects (font (size 1.27 1.27)) hide)
-    )
-    (property "MFR.Part #" "CL05B104KO5NNNC" (at 146.05 41.91 0)
-      (effects (font (size 1.27 1.27)) hide)
-    )
+    (property "LCSC" "C1525" (at 146.05 41.91 0)
+      (effects (font (size 1.27 1.27)) hide)
+    )
+    (property "MFR. Part#" "CL05B104KO5NNNC" (at 146.05 41.91 0)
+      (effects (font (size 1.27 1.27)) hide)
+    )
