File: hardware/moco-oi401/moco-oi401.kicad_pcb (KiCad board)
At the start: 2 copper layers, 40 x 40 mm, 75 parts, among them J1 Debug, J2 Serial, J3 V+, J4 V-, J5 A, J6 B, J7 C, SW1 RESET, U1 RT9013-33GB, U2 STM32G431CBUx, U3 DRV8316CR, U4 LM4040A50, U5 AS5047x, Y1 8MHz

Commit message: Update part#
Parts:
- C13: value 47nF/100V -> 47nF/50V
- R2: value 5k -> 5.1k
- Y1: value 8MHz -> 16MHz
Routing:
- net GNDPWR: vias 20 -> 22
- net GND: vias 51 -> 60
Other:
- board text added: "SB1: 3.3V LDO Bypass SB2: nSLEEP Reset SB3: V_{REF} Selection"
