File: hardware/moco-oi401/moco-oi401.kicad_sch (KiCad schematic)
At the start: 20 parts, among them J1 Debug, J2 Serial, J3 V+, J4 V-, U1 RT9013-33GB

Commit message: Rename "OI451" to "OI401"
Other:
- title: moco-OI451 -> moco-OI401
Changed lines of the file:
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@@
   (paper "A4")
   (title_block
-    (title "moco-OI451")
+    (title "moco-OI401")
     (rev "1.0")
     (comment 1 "BLDC motor controller/driver")
@@
     )
     (instances
-      (project "moco-oi451"
+      (project "moco-oi401"
         (path "/171831cd-2a0d-47b9-8420-65898c688d08"
           (reference "H3") (unit 1)
@@
     (pin "1")
     (instances
-      (project "moco-oi451"
+      (project "moco-oi401"
         (path "/171831cd-2a0d-47b9-8420-65898c688d08"
           (reference "#PWR011") (unit 1)
@@
     (pin "1")
     (instances
-      (project "moco-oi451"
+      (project "moco-oi401"
         (path "/171831cd-2a0d-47b9-8420-65898c688d08"
           (reference "#PWR05") (unit 1)
@@
     (pin "1")
     (instances
-      (project "moco-oi451"
+      (project "moco-oi401"
         (path "/171831cd-2a0d-47b9-8420-65898c688d08"
           (reference "#PWR03") (unit 1)
@@
     (pin "2")
     (instances
-      (project "moco-oi451"
+      (project "moco-oi401"
         (path "/171831cd-2a0d-47b9-8420-65898c688d08"
           (reference "R2") (unit 1)
@@
     (pin "1")
     (instances
-      (project "moco-oi451"
+      (project "moco-oi401"
         (path "/171831cd-2a0d-47b9-8420-65898c688d08"
           (reference "#PWR08") (unit 1)
@@
     (pin "1")
     (instances
-      (project "moco-oi451"
+      (project "moco-oi401"
         (path "/171831cd-2a0d-47b9-8420-65898c688d08"
           (reference "#PWR04") (unit 1)
@@
     (pin "3")
     (instances
-      (project "moco-oi451"
+      (project "moco-oi401"
         (path "/171831cd-2a0d-47b9-8420-65898c688d08"
           (reference "J2") (unit 1)
@@
     (pin "1")
     (instances
-      (project "moco-oi451"
+      (project "moco-oi401"
         (path "/171831cd-2a0d-47b9-8420-65898c688d08"
           (reference "TP3") (unit 1)
@@
     (pin "1")
     (instances
-      (project "moco-oi451"
+      (project "moco-oi401"
         (path "/171831cd-2a0d-47b9-8420-65898c688d08"
           (reference "#PWR01") (unit 1)
@@
     (pin "1")
     (instances
-      (project "moco-oi451"
+      (project "moco-oi401"
         (path "/171831cd-2a0d-47b9-8420-65898c688d08"
           (reference "#PWR02") (unit 1)
@@
     (pin "1")
     (instances
-      (project "moco-oi451"
+      (project "moco-oi401"
         (path "/171831cd-2a0d-47b9-8420-65898c688d08"
           (reference "#PWR012") (unit 1)
@@
     (pin "1")
     (instances
-      (project "moco-oi451"
+      (project "moco-oi401"
         (path "/171831cd-2a0d-47b9-8420-65898c688d08"
           (reference "#PWR09") (unit 1)
@@
     (pin "1")
     (instances
-      (project "moco-oi451"
+      (project "moco-oi401"
         (path "/171831cd-2a0d-47b9-8420-65898c688d08"
           (reference "TP1") (unit 1)
@@
     (pin "2")
     (instances
-      (project "moco-oi451"
+      (project "moco-oi401"
         (path "/171831cd-2a0d-47b9-8420-65898c688d08"
           (reference "R3") (unit 1)
@@
     (pin "2")
     (instances
-      (project "moco-oi451"
+      (project "moco-oi401"
         (path "/171831cd-2a0d-47b9-8420-65898c688d08"
           (reference "SB2") (unit 1)
@@
     (pin "2")
     (instances
-      (project "moco-oi451"
+      (project "moco-oi401"
         (path "/171831cd-2a0d-47b9-8420-65898c688d08"
           (reference "C1") (unit 1)
@@
     (pin "5")
     (instances
-      (project "moco-oi451"
+      (project "moco-oi401"
         (path "/171831cd-2a0d-47b9-8420-65898c688d08"
           (reference "U1") (unit 1)
@@
     (pin "2")
     (instances
-      (project "moco-oi451"
+      (project "moco-oi401"
         (path "/171831cd-2a0d-47b9-8420-65898c688d08"
           (reference "R1") (unit 1)
@@
     (pin "4")
     (instances
-      (project "moco-oi451"
+      (project "moco-oi401"
         (path "/171831cd-2a0d-47b9-8420-65898c688d08"
           (reference "LD1") (unit 1)
@@
     (pin "1")
     (instances
-      (project "moco-oi451"
+      (project "moco-oi401"
         (path "/171831cd-2a0d-47b9-8420-65898c688d08"
           (reference "J3") (unit 1)
@@
     (pin "1")
     (instances
-      (project "moco-oi451"
+      (project "moco-oi401"
         (path "/171831cd-2a0d-47b9-8420-65898c688d08"
           (reference "TP2") (unit 1)
@@
     )
     (instances
-      (project "moco-oi451"
+      (project "moco-oi401"
         (path "/171831cd-2a0d-47b9-8420-65898c688d08"
           (reference "H2") (unit 1)
@@
     (pin "1")
     (instances
-      (project "moco-oi451"
+      (project "moco-oi401"
         (path "/171831cd-2a0d-47b9-8420-65898c688d08/8c626c9e-bc00-4eb5-9b1c-4380247b0f28"
           (reference "#PWR?") (unit 1)
@@
     )
     (instances
-      (project "moco-oi451"
+      (project "moco-oi401"
         (path "/171831cd-2a0d-47b9-8420-65898c688d08"
           (reference "H1") (unit 1)
@@
     (pin "1")
     (instances
-      (project "moco-oi451"
+      (project "moco-oi401"
         (path "/171831cd-2a0d-47b9-8420-65898c688d08/e49edf63-a462-4dde-9ddc-a334d0522771"
           (reference "#PWR?") (unit 1)
@@
     (pin "2")
     (instances
-      (project "moco-oi451"
+      (project "moco-oi401"
         (path "/171831cd-2a0d-47b9-8420-65898c688d08"
           (reference "C2") (unit 1)
@@
     (pin "8")
     (instances
-      (project "moco-oi451"
+      (project "moco-oi401"
         (path "/171831cd-2a0d-47b9-8420-65898c688d08"
           (reference "J1") (unit 1)
@@
     (pin "1")
     (instances
-      (project "moco-oi451"
+      (project "moco-oi401"
         (path "/171831cd-2a0d-47b9-8420-65898c688d08"
           (reference "#PWR013") (unit 1)
@@
     (pin "1")
     (instances
-      (project "moco-oi451"
+      (project "moco-oi401"
         (path "/171831cd-2a0d-47b9-8420-65898c688d08"
           (reference "J4") (unit 1)
@@
     (pin "2")
     (instances
-      (project "moco-oi451"
+      (project "moco-oi401"
         (path "/171831cd-2a0d-47b9-8420-65898c688d08/e49edf63-a462-4dde-9ddc-a334d0522771"
           (reference "NT?") (unit 1)
@@
     (pin "2")
     (instances
-      (project "moco-oi451"
+      (project "moco-oi401"
         (path "/171831cd-2a0d-47b9-8420-65898c688d08"
           (reference "SB1") (unit 1)
@@
     (pin "1")
     (instances
-      (project "moco-oi451"
+      (project "moco-oi401"
         (path "/171831cd-2a0d-47b9-8420-65898c688d08"
           (reference "#PWR07") (unit 1)
@@
     )
     (instances
-      (project "moco-oi451"
+      (project "moco-oi401"
         (path "/171831cd-2a0d-47b9-8420-65898c688d08" (page "4"))
       )
@@
     )
     (instances
-      (project "moco-oi451"
+      (project "moco-oi401"
         (path "/171831cd-2a0d-47b9-8420-65898c688d08" (page "2"))
       )
@@
     )
     (instances
-      (project "moco-oi451"
+      (project "moco-oi401"
         (path "/171831cd-2a0d-47b9-8420-65898c688d08" (page "3"))
       )

Commit message: Update part#
Parts:
- C1, C2: LCSC (none) -> C15849; MFR. Part# (none) -> CL10A105KB8NNNC
- J2: LCSC (none) -> C514175; MFR. Part# (none) -> SM03B-GHS-TB(LF)(SN)
- LD1: JLCPCB Part # C375569 -> (none); LCSC (none) -> C375569; MFR. Part# (none) -> E6C0606RGBC3UDA; MFR.Part # E6C0606RGBC3UDA -> (none)
- R1: JLCPCB Part # C25130 -> (none); LCSC (none) -> C25104; MFR. Part# (none) -> 0402WGF3300TCE; MFR.Part # 0402WGF6800TCE -> (none)
- R2: value 5k -> 5.1k; JLCPCB Part # C11702 -> (none); LCSC (none) -> C25905; MFR. Part# (none) -> 0402WGF5101TCE; MFR.Part # 0402WGF1001TCE -> (none)
- R3: JLCPCB Part # C25104 -> (none); LCSC (none) -> C25104; MFR. Part# (none) -> 0402WGF3300TCE; MFR.Part # 0402WGF3300TCE -> (none)
- U1: LCSC (none) -> C587158; MFR. Part# (none) -> TPRT9013-33GB
Connections:
- no-connect marks 6 -> 11
Other:
- note added: "+10V~35V"
- moved on the sheet: J1, J2, J3, J4, LD1, R1, R2, R3, TP3
