File: hardware/moco-oi401/rotary_sensor.kicad_sch (KiCad schematic)
At the start: 2 parts, among them U5 AS5047x

Commit message: Update part#
Parts:
- C34: LCSC (none) -> C14663; MFR. Part# (none) -> CC0603KRX7R9BB104
- U5: JLCPCB Part # C962063 -> (none); LCSC (none) -> C962063; MFR. Part# (none) -> AS5047P-ATSM; MFR.Part # AS5047P-ATSM -> (none)
Changed lines of the file:
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@@
       (effects (font (size 1.27 1.27)) hide)
     )
-    (property "JLCPCB Part #" "C962063" (at 143.51 100.33 0)
+    (property "LCSC" "C962063" (at 143.51 100.33 0)
       (effects (font (size 1.27 1.27)) hide)
     )
-    (property "MFR.Part #" "AS5047P-ATSM" (at 143.51 100.33 0)
+    (property "MFR. Part#" "AS5047P-ATSM" (at 143.51 100.33 0)
       (effects (font (size 1.27 1.27)) hide)
     )
@@
       (effects (font (size 1.27 1.27)) hide)
     )
+    (property "LCSC" "C14663" (at 133.35 82.55 0)
+      (effects (font (size 1.27 1.27)) hide)
+    )
+    (property "MFR. Part#" "CC0603KRX7R9BB104" (at 133.35 82.55 0)
+      (effects (font (size 1.27 1.27)) hide)
+    )
