File: hardware/moco-bkd8316/moco-bkd8316.kicad_pcb (KiCad board)
At the start: 2 copper layers, 50 x 45 mm, 57 parts, among them J1 Conn_01x02, J2 Conn_02x10_Odd_Even, J3 Conn_01x01, J4 Conn_01x01, J5 Conn_01x01, U1 RT9013-33GB, U2 DRV8316CR, U3 LM4040D33FTA

Commit message: BKD8316 routed
Parts:
- removed C19, C20, C21, C22, C23, C24: 22uF/50V, Capacitor_SMD:C_0805_2012Metric
- removed R11, R12: 330R, Resistor_SMD:R_0603_1608Metric
- removed SB2: SolderJumper_2_Bridged, Jumper:SolderJumper-2_P1.3mm_Bridged_RoundedPad1.0x1.5mm
- removed TP5: V_{SLEEP}, TestPoint:TestPoint_Pad_D1.0mm
- removed U2: DRV8316CR, moco:VQFN-40_RGF_5x7mm_0.5mm_pitch_thermalpad
- removed U3: LM4040D33FTA, Package_TO_SOT_SMD:SOT-23
- added D1: LM4040A50, Package_TO_SOT_SMD:SOT-353_SC-70-5, F.Cu at (145.4, 96.5)
- added J6: B, moco:wire_3.2mm, F.Cu at (162.0, 110.0)
- added J7: C, moco:wire_3.2mm, F.Cu at (162.0, 102.0)
- added NT1: NetTie_2, NetTie:NetTie-2_SMD_Pad0.5mm, F.Cu at (142.3, 125.8)
- added SW1: RESET, Button_Switch_SMD:SW_SPST_CK_RS282G05A3, F.Cu at (148.2, 92.0)
- C10, C9: value 1uF -> 22pF
- C11, C12: value 22pF -> 10uF/50V; footprint Capacitor_SMD:C_0603_1608Metric -> Capacitor_SMD:C_0805_2012Metric
- C13: value 22pF -> 10uF/50V; footprint Capacitor_SMD:C_0603_1608Metric -> Capacitor_SMD:C_0805_2012Metric; moved to B.Cu
- C14: value 47uF/50V -> 10uF/50V; footprint Capacitor_SMD:CP_Elec_6.3x7.7 -> Capacitor_SMD:C_0805_2012Metric
- C15: value 22uF/50V -> 10uF/50V
- C16, C17, C18: value 22uF/50V -> 10uF/50V; moved to B.Cu
- C5: value 100nF/50V -> 10uF/50V; footprint Capacitor_SMD:C_0603_1608Metric -> Capacitor_SMD:C_0805_2012Metric
- C6: value 10uF/50V -> 100nF/6.3V; footprint Capacitor_SMD:C_0805_2012Metric -> Capacitor_SMD:C_0603_1608Metric
- C7: value 100nF/6.3V -> 22uF/16V; footprint Capacitor_SMD:C_0603_1608Metric -> Capacitor_SMD:C_0805_2012Metric
- C8: value 22uF -> 22pF
- J1: value Conn_01x02 -> Conn_02x10_Odd_Even; footprint Connector_AMASS:AMASS_XT30UPB-M_1x02_P5.0mm_Vertical -> Connector_PinSocket_2.54mm:PinSocket_2x10_P2.54mm_Vertical
- J2: value Conn_02x10_Odd_Even -> Conn_01x02; footprint Connector_PinSocket_2.54mm:PinSocket_2x10_P2.54mm_Vertical -> Connector_PinHeader_2.54mm:PinHeader_1x02_P2.54mm_Vertical
- J3, J4, J5: value Conn_01x01 -> A
- L1: footprint Inductor_SMD:L_Taiyo-Yuden_NR-50xx -> Inductor_SMD:L_Taiyo-Yuden_MD-3030
- R1: value 1.5k -> 22R
- R10: value 330R -> 10k
- R2: value DNI -> 5.1k
- R3: value 22R -> 5.1k
- R4: value DNI -> 330R
- R5, R6: value 10k -> 330R
- R7: value 2.7k -> 1.5k
- R8: value 10k -> 10k/100mW
- R9: value 2.7k -> 10k
- TP1: value V_{DD} -> TestPoint; footprint TestPoint:TestPoint_Pad_D1.0mm -> TestPoint:TestPoint_Pad_D1.5mm
- TP2: value V_{DR} -> TestPoint; footprint TestPoint:TestPoint_Pad_D1.0mm -> TestPoint:TestPoint_Pad_D1.5mm
- TP3: value V_{BK} -> TestPoint; footprint TestPoint:TestPoint_Pad_D1.0mm -> TestPoint:TestPoint_Pad_D1.5mm
- TP4: value V_{CC} -> nSLEEP
- U1: value RT9013-33GB -> DRV8316CR; footprint Package_TO_SOT_SMD:SOT-23-5 -> moco:VQFN-40_RGF_5x7mm_0.5mm_pitch_thermalpad
- moved TP3 59.1 mm to (139.5, 93.0)
- moved TP2 56.0 mm to (139.7, 118.7)
- moved TP1 55.6 mm to (142.7, 96.4)
- moved TP4 51.9 mm to (153.2, 96.5)
- moved J2 38.3 mm to (143.5, 128.3), turned to 180 degrees
- moved J1 30.6 mm to (133.8, 98.6)
- moved J3 21.4 mm to (148.0, 127.1), turned to 90 degrees
- moved C13 20.7 mm to (152.5, 119.8)
- moved R1 19.3 mm to (144.9, 118.0)
- moved R10 19.1 mm to (151.2, 96.5), turned to -90 degrees
- moved LD1 18.0 mm to (142.0, 119.8), turned to 90 degrees
- moved C12 17.8 mm to (152.5, 120.8)
- moved R7 17.4 mm to (144.8, 120.8), turned to 0 degrees
- moved R3 16.3 mm to (151.5, 104.5), turned to -90 degrees
- moved R5 15.7 mm to (141.2, 113.5), turned to 0 degrees
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- renumbered H4 to H1, H3 to H2, H2 to H3, H1 to H4
Connections:
- C1 pad 1: Net-(U2-CPL) -> Net-(U1-CPL)
- C1 pad 2: Net-(U2-CPH) -> Net-(U1-CPH)
- C10 pad 1: VCC -> SOC
- C11 pad 1: SO_A -> VBUS
- C11 pad 2: GND -> GNDPWR
- C12 pad 1: SO_B -> VBUS
- C12 pad 2: GND -> GNDPWR
- C13 pad 1: SO_C -> VBUS
- C13 pad 2: GND -> GNDPWR
- C14 pad 1: Vdrive -> VBUS
- C14 pad 2: GND -> GNDPWR
- C15 pad 1: Vdrive -> VBUS
- C15 pad 2: GND -> GNDPWR
- C16 pad 1: Vdrive -> VBUS
- C16 pad 2: GND -> GNDPWR
- C17 pad 1: Vdrive -> VBUS
- C17 pad 2: GND -> GNDPWR
- C18 pad 1: Vdrive -> VBUS
- C18 pad 2: GND -> GNDPWR
- C2 pad 1: Net-(U2-CP) -> Net-(U1-CP)
- C2 pad 2: Vdrive -> VBUS
- C3 pad 2: VDD -> +3.3V
- C4 pad 1: GND -> GNDPWR
- C4 pad 2: Vdrive -> VBUS
- C5 pad 1: GND -> GNDPWR
- C5 pad 2: Vdrive -> VBUS
- C6 pad 1: GND -> VREF
- C6 pad 2: Vdrive -> GND
- C7 pad 1: Net-(SB2-A) -> GND
- C7 pad 2: GND -> VCC
- C8 pad 1: GND -> SOA
- C8 pad 2: Net-(SB1-A) -> GND
- C9 pad 1: Net-(SB1-A) -> SOB
- J1 pad 1: GND -> VCC
- J1 pad 2: Vdrive -> +3.3V
- J2 pad 1: VCC -> VBUS
- J2 pad 2: GND -> GNDPWR
- J3 pad 1: /OUT_B -> VBUS
- J4 pad 1: /OUT_A -> GNDPWR
- J5 pad 1: /OUT_C -> /OUTA
- L1 pad 1: Net-(U2-SW_BK) -> Net-(U1-SW_BK)
- L1 pad 2: Net-(SB1-A) -> VCC
- R1 pad 1: Net-(LD1-K) -> Net-(U1-SW_BK)
- R1 pad 2: GND -> VCC
- R10 pad 1: SO_A -> Net-(R10-Pad1)
- R10 pad 2: Net-(U2-SOA) -> ~{SLEEP}
- R2 pad 1: VDD -> +3.3V
- R2 pad 2: Net-(SB2-A) -> MISO
- R3 pad 1: Net-(U2-SW_BK) -> +3.3V
- R3 pad 2: Net-(SB1-A) -> ~{FAULT}
- R4 pad 1: Net-(SB2-A) -> SOA
- R4 pad 2: GND -> Net-(U1-SOA)
- R5 pad 1: VCC -> SOB
- R5 pad 2: ~{FAULT} -> Net-(U1-SOB)
- R6 pad 1: VCC -> SOC
- R6 pad 2: SPI_MISO -> Net-(U1-SOC)
- R7 pad 1: Vdrive -> Net-(LD1-K)
- R7 pad 2: Net-(U3-K) -> GND
- R8 pad 1: Net-(U3-K) -> VBUS
- R9 pad 2: ~{SLEEP} -> Net-(R10-Pad1)
- SB1 pad 1: Net-(SB1-A) -> VREF
- SB1 pad 2: VCC -> +3.3V
- TP1 pad 1: VDD -> +3.3V
- TP2 pad 1: Vdrive -> VCC
- TP3 pad 1: Net-(SB1-A) -> GND
- TP4 pad 1: VCC -> ~{SLEEP}
- U1 pad 1: Net-(SB1-A) -> unconnected-(U1-NC-Pad1)
- U1 pad 3: Net-(SB1-A) -> VCC
- U1 pad 4: unconnected-(U1-NC-Pad4) -> GND
- U1 pad 5: VCC -> Net-(U1-SW_BK)
Routing:
- net VCC: track 0.00 -> 58.5 mm, vias 0 -> 2
- net VBUS: track 0.00 -> 51.3 mm, vias 0 -> 15
- net +3.3V: track 0.00 -> 40.1 mm, vias 0 -> 4
- net ~{CS}: track 0.00 -> 29.3 mm, vias 0 -> 1
- net DRVOFF: track 0.00 -> 29.1 mm
- net ~{FAULT}: track 0.00 -> 25.8 mm
- net GND: track 0.00 -> 24.6 mm, vias 0 -> 53
- net SCLK: track 0.00 -> 23.5 mm, vias 0 -> 1
- net ~{SLEEP}: track 0.00 -> 23.0 mm, vias 0 -> 2
- net PWM_H_A: track 0.00 -> 23.0 mm
- net PWM_H_B: track 0.00 -> 22.3 mm
- net PWM_H_C: track 0.00 -> 21.6 mm
- net MOSI: track 0.00 -> 20.9 mm
- net PWM_L_A: track 0.00 -> 19.6 mm
- net MISO: track 0.00 -> 19.0 mm
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- added copper zone on F.Cu, net /OUTA
- added copper zone on F.Cu, net /OUTB
- added copper zone on F.Cu, net /OUTC
- added copper zone on B.Cu, net GND
- added copper zone on F.Cu, net GND
- added copper zone on B.Cu, net GNDPWR
- added copper zone on F.Cu, net GNDPWR
- added copper zone on B.Cu, net VBUS
- added copper zone on F.Cu, net VBUS
Other:
- board size 50 x 45 mm -> 35.5 x 41 mm
- board text added: "${TITLE}"
- board text added: "+"
- board text added: "-"
- board text added: "1"
- board text added: "10~35V"
- board text added: "19"
- board text added: "2"
- board text added: "20"
- board text added: "A"
- board text added: "B"
- board text added: "C"
- board text added: "VCC"
- board text added: "v${REVISION}"
