File: hardware/moco-bkd8316/moco-bkd8316.kicad_sch (KiCad schematic)
At the start: 57 parts, among them J1 Conn_01x02, J2 Conn_02x10_Odd_Even, J3 Conn_01x01, J4 Conn_01x01, J5 Conn_01x01, U1 RT9013-33GB, U2 DRV8316CR, U3 LM4040D33FTA

Commit message: Rename "moco8316" to "moco-bkd8316"
Other:
- title: (none) -> moco-BKD8316

Commit message: BKD8316 routed
Parts:
- removed C1: 47nF/50V, Capacitor_SMD:C_0603_1608Metric, symbol Device:C_Small
- removed C10, C9: 1uF, Capacitor_SMD:C_0603_1608Metric, symbol Device:C
- removed C11, C12, C13: 22pF, Capacitor_SMD:C_0603_1608Metric, symbol Device:C
- removed C14: 47uF/50V, Capacitor_SMD:CP_Elec_6.3x7.7, symbol Device:C_Polarized
- removed C15, C16, C17, C18, C19, C20, C21, C22, C23, C24: 22uF/50V, Capacitor_SMD:C_0805_2012Metric, symbol Device:C
- removed C2: 1uF/16V, Capacitor_SMD:C_0603_1608Metric, symbol Device:C_Small
- removed C3: 1uF/6.3V, Capacitor_SMD:C_0603_1608Metric, symbol Device:C_Small
- removed C4, C5: 100nF/50V, Capacitor_SMD:C_0603_1608Metric, symbol Device:C_Small
- removed C6: 10uF/50V, Capacitor_SMD:C_0805_2012Metric, symbol Device:C_Small
- removed C7: 100nF/6.3V, Capacitor_SMD:C_0603_1608Metric, symbol Device:C
- removed C8: 22uF, Capacitor_SMD:C_0603_1608Metric, symbol Device:C_Small
- removed J1: Conn_01x02, Connector_AMASS:AMASS_XT30UPB-M_1x02_P5.0mm_Vertical, symbol Connector_Generic:Conn_01x02
- removed J2: Conn_02x10_Odd_Even, Connector_PinSocket_2.54mm:PinSocket_2x10_P2.54mm_Vertical, symbol Connector_Generic:Conn_02x10_Odd_Even
- removed J3, J4, J5: Conn_01x01, moco:wire_3.2mm, symbol Connector_Generic:Conn_01x01
- removed L1: 47uH, Inductor_SMD:L_Taiyo-Yuden_NR-50xx, symbol Device:L
- removed R1: 1.5k, Resistor_SMD:R_0603_1608Metric, symbol Device:R
- removed R10, R11, R12: 330R, Resistor_SMD:R_0603_1608Metric, symbol Device:R
- removed R2, R4: DNI, Resistor_SMD:R_0603_1608Metric, symbol Device:R
- removed R3: 22R, Resistor_SMD:R_0603_1608Metric, symbol Device:R
- removed R5, R6, R8: 10k, Resistor_SMD:R_0603_1608Metric, symbol Device:R
- removed R9: 2.7k, Resistor_SMD:R_0603_1608Metric, symbol Device:R
- removed SB1: SolderJumper_2_Open, Jumper:SolderJumper-2_P1.3mm_Open_RoundedPad1.0x1.5mm, symbol Jumper:SolderJumper_2_Open
- removed SB2: SolderJumper_2_Bridged, Jumper:SolderJumper-2_P1.3mm_Bridged_RoundedPad1.0x1.5mm, symbol Jumper:SolderJumper_2_Bridged
- removed TP3: V_{BK}, TestPoint:TestPoint_Pad_D1.0mm, symbol Connector:TestPoint
- removed TP4: V_{CC}, TestPoint:TestPoint_Pad_D1.0mm, symbol Connector:TestPoint
- removed TP5: V_{SLEEP}, TestPoint:TestPoint_Pad_D1.0mm, symbol Connector:TestPoint
- removed U1: RT9013-33GB, Package_TO_SOT_SMD:SOT-23-5, symbol rp-micro:RT9013-33GB
- removed U2: DRV8316CR, moco:VQFN-40_RGF_5x7mm_0.5mm_pitch_thermalpad, symbol moco8316:DRV8316CR
- removed U3: LM4040D33FTA, Package_TO_SOT_SMD:SOT-23, symbol Reference_Voltage:LM4040DBZ-3
- added C? (x3): 22pF, Capacitor_SMD:C_0603_1608Metric, symbol Device:C
- added C? (x8): 10uF/50V, Capacitor_SMD:C_0805_2012Metric, symbol Device:C
- added C?: 22uF/16V, Capacitor_SMD:C_0805_2012Metric, symbol Device:C_Small
- added C?: 47nF/50V, Capacitor_SMD:C_0603_1608Metric, symbol Device:C_Small
- added C?: 100nF/6.3V, Capacitor_SMD:C_0603_1608Metric, symbol Device:C
- added C?: 10uF/50V, Capacitor_SMD:C_0805_2012Metric, symbol Device:C_Small
- added C?: 100nF/50V, Capacitor_SMD:C_0603_1608Metric, symbol Device:C_Small
- added C?: 1uF/16V, Capacitor_SMD:C_0603_1608Metric, symbol Device:C_Small
- added C?: 1uF/6.3V, Capacitor_SMD:C_0603_1608Metric, symbol Device:C_Small
- added J1: Conn_02x10_Odd_Even, Connector_PinSocket_2.54mm:PinSocket_2x10_P2.54mm_Vertical, symbol Connector_Generic:Conn_02x10_Odd_Even
- added J2: Conn_01x02, Connector_PinHeader_2.54mm:PinHeader_1x02_P2.54mm_Vertical, symbol Connector_Generic:Conn_01x02
- added J? (x3): A, moco:wire_3.2mm, symbol Connector_Generic:Conn_01x01
- added J?: C, moco:wire_3.2mm, symbol Connector_Generic:Conn_01x01
- added J?: B, moco:wire_3.2mm, symbol Connector_Generic:Conn_01x01
- added L?: 47uH, Inductor_SMD:L_Taiyo-Yuden_MD-3030, symbol Device:L
- added NT?: NetTie_2, NetTie:NetTie-2_SMD_Pad0.5mm, symbol Device:NetTie_2
- added R? (x2): 5.1k, Resistor_SMD:R_0603_1608Metric, symbol Device:R
- added R? (x3): 330R, Resistor_SMD:R_0603_1608Metric, symbol Device:R
- added R?: 10k/100mW, Resistor_SMD:R_0603_1608Metric, symbol Device:R
- added R?: 22R, Resistor_SMD:R_0603_1608Metric, symbol Device:R
- added R? (x2): 10k, Resistor_SMD:R_0603_1608Metric, symbol Device:R
- added SB2: SolderJumper_2_Open, Jumper:SolderJumper-2_P1.3mm_Open_RoundedPad1.0x1.5mm, symbol Jumper:SolderJumper_2_Open
- added SW1: RESET, Button_Switch_SMD:SW_SPST_CK_RS282G05A3, symbol Switch:SW_Push
- added TP3: TestPoint, TestPoint:TestPoint_Pad_D1.5mm, symbol Connector:TestPoint
- added TP3: nSLEEP, TestPoint:TestPoint_Pad_D1.0mm, symbol Connector:TestPoint
- added U4: LM4040A50, Package_TO_SOT_SMD:SOT-353_SC-70-5, symbol Reference_Voltage:LM4040DCK-5
- added U?: DRV8316CR, moco:VQFN-40_RGF_5x7mm_0.5mm_pitch_thermalpad, symbol moco8316:DRV8316CR
- R7: value 2.7k -> 1.5k
- TP1: value V_{DD} -> TestPoint; footprint TestPoint:TestPoint_Pad_D1.0mm -> TestPoint:TestPoint_Pad_D1.5mm
- TP2: value V_{DR} -> TestPoint; footprint TestPoint:TestPoint_Pad_D1.0mm -> TestPoint:TestPoint_Pad_D1.5mm
- renumbered H4 to H1, H3 to H2, H2 to H3, H1 to H4
Connections:
- net DRVOFF: now also J1.4 (Pin_4), U?.21 (DRVOFF)
- net GND: now also R7.2, C?.1, C?.1, C?.2, C?.2, C?.2, C?.2, J1.19 (Pin_19), J1.20 (Pin_20), NT?.1, SW1.1, TP3.1, U4.1 (A), U?.2 (AGND), U?.26 (AGND), U?.4 (GND_BK), U?.41 (EP)
- net PWM_H_A: now also J1.6 (Pin_6), U?.27 (INHA)
- net PWM_H_B: now also J1.8 (Pin_8), U?.29 (INHB)
- net PWM_H_C: now also J1.10 (Pin_10), U?.31 (INHC)
- net PWM_L_A: now also J1.5 (Pin_5), U?.28 (INLA)
- net PWM_L_B: now also J1.7 (Pin_7), U?.30 (INLB)
- net PWM_L_C: now also J1.9 (Pin_9), U?.32 (INLC)
- net VCC: now also TP2.1, C?.2, J1.1 (Pin_1), L?.2, R?.2, U?.3 (FB_BK)
- net ~{FAULT}: now also J1.3 (Pin_3), R?.2, U?.22 (nFAULT)
- net ~{SLEEP}: now also R?.2, SW1.2, TP3.1, U?.23 (nSLEEP)
- net at LD1.1 (K): now also R7.1
- net VDD renamed +3.3V
- net +3.3V: now also C?.2, J1.2 (Pin_2), R?.1, R?.1, SB2.2 (B), U?.25 (AVDD)
- removed net Vdrive: R7.1, TP2.1
- new net: R?.2, U?.39 (SOB)
- new net: C?.1, U?.6 (CPL)
- new net: C?.2, U?.7 (CPH)
- new net: R?.1, R?.2, U4.3 (K)
- new net: L?.1, R?.1, U?.5 (SW_BK)
- new net: R?.1, R?.2
- new net: R?.2, U?.38 (SOC)
- new net: R?.2, U?.40 (SOA)
- new net: C?.1, U?.8 (CP)
- new net GNDPWR: C?.1, C?.1, C?.2, C?.2, C?.2, C?.2, C?.2, C?.2, C?.2, C?.2, J2.2 (Pin_2), J?.1 (Pin_1), NT?.2, U?.12 (PGND), U?.15 (PGND), U?.18 (PGND)
- new net MISO: J1.12 (Pin_12), R?.2, U?.33 (SDO)
- new net MOSI: J1.14 (Pin_14), U?.34 (SDI)
- new net OUTA: J?.1 (Pin_1), U?.13 (OUTA), U?.14 (OUTA)
- new net OUTB: J?.1 (Pin_1), U?.16 (OUTB), U?.17 (OUTB)
- new net OUTC: J?.1 (Pin_1), U?.19 (OUTC), U?.20 (OUTC)
- new net SCLK: J1.16 (Pin_16), U?.35 (SCLK)
- new net SOA: C?.1, J1.17 (Pin_17), R?.1
- new net SOB: C?.1, J1.15 (Pin_15), R?.1
- new net SOC: C?.1, J1.13 (Pin_13), R?.1
- new net VBUS: C?.1, C?.1, C?.1, C?.1, C?.1, C?.1, C?.1, C?.1, C?.2, C?.2, C?.2, J2.1 (Pin_1), J?.1 (Pin_1), R?.1, U?.10 (VM), U?.11 (VM), U?.9 (VM)
- new net VREF: C?.1, J1.11 (Pin_11), SB2.1 (A), U?.37 (VREF/LILM)
- new net ~{CS}: J1.18 (Pin_18), U?.36 (nSCS)
Other:
- note added: "Bulk Capacitors"
- note added: "SPI: - Mode=1 * CPOL=0(Clock is low when idle) * CPHA=1(Data sampled on falling edge) - 16-bit data - MSB first - nSCS pin active low - 5MHz clock"
- note added: "VM operating voltage: 4.5V~35V"
- note added: "V_{S}=10V~35V V_{Z}=5V I_{Z}=65uA~15mA I_{L}=10uA~30uA Rs: 1.99kohm~38.46kohm"
- note added: "nSLEEP ON"
- note added: "nSLEEP pin: Input logic high current @ 5V: 10~30 uA Input logic high voltage: 1.6~5.5 V Input pulldown resistance: 150~300 kohm, typ. 200"
- note removed: "Buck capacitance"
- note removed: "nSLEEP pin: Input logic high current @ 5V: 10~30 uA Input logic high voltage: 1.6~5.5 V"
