File: hardware/moco-rd401/moco-rd401.kicad_pcb (KiCad board)
At the start: 4 copper layers, 32 x 32 mm, 93 parts, among them J1 I^{2}C, J2 Serial, J3 Debug, J4 V+, J5 V-, J6 U, J7 V, J8 W, Q1 SiZ250DT, Q2 SiZ250DT, Q3 SiZ250DT, SW1 RESET, U1 STSPIN32F0A, U2 MA702

Commit message: Routed
Parts:
- removed the R3 at (150.6, 90.7)
- added C26: 10uF/50V, Capacitor_SMD:C_0805_2012Metric, B.Cu at (158.8, 111.9)
- added C27: 10uF/50V, Capacitor_SMD:C_0805_2012Metric, B.Cu at (158.8, 109.9)
- added C28: 10uF/50V, Capacitor_SMD:C_0805_2012Metric, B.Cu at (158.8, 113.9)
- moved R4 3.00 mm to (139.5, 93.4), turned to 0 degrees
- moved NT1 2.42 mm to (156.7, 110.5)
- moved TP2 1.85 mm to (141.9, 94.9)
- moved TP3 1.10 mm to (141.1, 109.0)
- moved D1 0.60 mm to (144.2, 105.2)
- moved J4 0.36 mm to (161.9, 86.1)
- moved J5 0.36 mm to (156.9, 86.1)
- moved SW1 0.18 mm to (139.6, 90.8)
- turned R17 to -90 degrees
- turned R3 to 90 degrees
- renumbered C27 to C25, C26 to C29, R11 to R10, R12 to R11, R13 to R12, R14 to R13, R15 to R14, R16 to R15, R17 to R16, R18 to R17, R19 to R18, R20 to R19, R21 to R20, R22 to R21, R23 to R22, R24 to R23, R25 to R24, R26 to R25, R27 to R26, R28 to R27, R29 to R28, R30 to R29, R5 to R3, R31 to R30, R32 to R31, R33 to R32, R34 to R33, R6 to R4, R4 to R5, R7 to R6, R8 to R7, R9 to R8, R10 to R9, TP4 to TP3
Connections:
- J1 pad MP: unconnected-(J1-MountPin-PadMP) -> (no net)
- J2 pad MP: unconnected-(J2-MountPin-PadMP) -> (no net)
- J3 pad 2: /BOOT0 -> GND
- J3 pad 7: GND -> /~{RESET}
- U1 pad 42: /BOOT0 -> GND
Routing:
- net +3.3V: track 5.90 -> 61.8 mm, vias 0 -> 4
- net Vdrive: track 47.0 -> 97.0 mm, vias 39 -> 60
- net /USART1_TX: track 0.00 -> 38.7 mm, vias 0 -> 1
- net /USART1_RX: track 0.00 -> 29.5 mm, vias 0 -> 2
- net /~{RESET}: track 2.29 -> 27.9 mm, vias 0 -> 2
- net /I2C1_SDA: track 0.00 -> 21.5 mm, vias 0 -> 2
- net /I2C1_SCL: track 0.00 -> 19.8 mm, vias 0 -> 2
- net /Power Stage/RSU+: track 13.1 -> 30.8 mm, vias 2 -> 3
- net GND: track 10.6 -> 27.8 mm, vias 9 -> 39
- net /SPI_MISO: track 0.00 -> 15.4 mm, vias 0 -> 1
- net /SPI_SCLK: track 0.00 -> 14.7 mm, vias 0 -> 1
- net /USER_LED: track 0.00 -> 11.9 mm, vias 0 -> 2
- net +12V: track 2.44 -> 13.3 mm, vias 0 -> 1
- net Net-(U1F-OP2P): track 0.00 -> 10.7 mm, vias 0 -> 2
- net /SWCLK: track 0.00 -> 9.86 mm, vias 0 -> 1
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- added copper zone on B.Cu, net /Power Stage/OUTU
- added copper zone on B.Cu, net /Power Stage/OUTV
- added copper zone on B.Cu, net /Power Stage/OUTW
- added copper zone on In1.Cu, net GNDPWR
- added copper zone on In2.Cu, net GNDPWR
Other:
- outline, holes or cut-outs redrawn
- board text added: "${TITLE}"
- board text added: "+"
- board text added: "-"
- board text added: "1)SCL"
- board text added: "1)TX"
- board text added: "15~35V"
- board text added: "3.3V"
- board text added: "7"
- board text added: "8"
- board text added: "GND"
- board text added: "RX"
- board text added: "SDA"
- board text added: "U"
- board text added: "V"
- board text added: "W"
- board text added: "v${REVISION}"
