File: hardware/moco-rd401/moco-rd401.kicad_sch (KiCad schematic)
At the start: 35 parts, among them J1 I^{2}C, J2 Serial, J3 Debug, J4 V+, J5 V-, SW1 RESET, U1 STSPIN32F0A

Commit message: Routed
Parts:
- removed R3: 10k, Resistor_SMD:R_0402_1005Metric, symbol Device:R
- removed TP3: PF1, TestPoint:TestPoint_Pad_D1.0mm, symbol Connector:TestPoint
- J1, J2: symbol Connector_Generic_MountingPin:Conn_01x03_MountingPin -> Connector_Generic:Conn_01x03
- renumbered R5 to R3, R6 to R4, R4 to R5, TP4 to TP3
Connections:
- net BOOT0 is gone; now on net GND: J3.2 (Pin_2), U1.42 (BOOT0)
- net GND: no longer J3.7 (Pin_7)
- net ~{RESET}: now also J3.7 (Pin_7)
- no-connect marks 5 -> 3
