File: hardware/moco-rd401/power_stage.kicad_sch (KiCad schematic)
At the start: 63 parts, among them J6 U, J7 V, J8 W

Commit message: Routed
Parts:
- added C26, C27, C28: 10uF/50V, Capacitor_SMD:C_0805_2012Metric, symbol Device:C
- renumbered C27 to C25
Connections:
- net GNDPWR: now also C26.2, C27.2, C28.2
- net Vdrive: now also C26.1, C27.1, C28.1
Other:
- moved on the sheet: C16, C17, C18, C19, C20, C21, C22, C23, C24, C25
