File: hardware/moco-rd321/triple_half_bridge.kicad_sch (KiCad schematic)
At the start: 66 parts, among them J6 U, J7 V, J8 W

Commit message: Update readme
Connections:
- net OP1O: now also R?.2, U?.21 (OP1O); no longer R?.2, U?.47 (OP3O)
- net OP3O: now also R?.2, U?.47 (OP3O); no longer R?.2, U?.21 (OP1O)
Changed lines of the file:
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@@
   (junction (at 25.4 186.69) (diameter 0) (color 0 0 0 0)
   )
+  (junction (at 88.9 157.48) (diameter 0) (color 0 0 0 0)
+  )
+  (junction (at 114.3 157.48) (diameter 0) (color 0 0 0 0)
+  )
+  (junction (at 90.17 59.69) (diameter 0) (color 0 0 0 0)
+  )
+  (junction (at 203.2 44.45) (diameter 0) (color 0 0 0 0)
+  )
+  (junction (at 242.57 59.69) (diameter 0) (color 0 0 0 0)
+  )
+  (junction (at 213.36 120.65) (diameter 0) (color 0 0 0 0)
+  )
+  (junction (at 219.71 59.69) (diameter 0) (color 0 0 0 0)
+  )
+  (junction (at 101.6 157.48) (diameter 0) (color 0 0 0 0)
+  )
+  (junction (at 39.37 186.69) (diameter 0) (color 0 0 0 0)
+  )
+  (junction (at 67.31 67.31) (diameter 0) (color 0 0 0 0)
+  )
+  (junction (at 201.93 120.65) (diameter 0) (color 0 0 0 0)
+  )
+  (junction (at 52.07 186.69) (diameter 0) (color 0 0 0 0)
+  )
+  (junction (at 52.07 179.07) (diameter 0) (color 0 0 0 0)
+  )
+  (junction (at 50.8 165.1) (diameter 0) (color 0 0 0 0)
+  )
+  (junction (at 25.4 157.48) (diameter 0) (color 0 0 0 0)
+  )
+  (junction (at 25.4 165.1) (diameter 0) (color 0 0 0 0)
+  )
+  (junction (at 88.9 165.1) (diameter 0) (color 0 0 0 0)
+  )
+  (junction (at 90.17 124.46) (diameter 0) (color 0 0 0 0)
+  )
+  (junction (at 25.4 179.07) (diameter 0) (color 0 0 0 0)
+  )
+  (junction (at 101.6 165.1) (diameter 0) (color 0 0 0 0)
+  )
+  (junction (at 50.8 109.22) (diameter 0) (color 0 0 0 0)
+  )
   (junction (at 113.03 63.5) (diameter 0) (color 0 0 0 0)
   )
-  (junction (at 88.9 157.48) (diameter 0) (color 0 0 0 0)
-  )
-  (junction (at 114.3 157.48) (diameter 0) (color 0 0 0 0)
-  )
-  (junction (at 90.17 59.69) (diameter 0) (color 0 0 0 0)
-  )
-  (junction (at 203.2 44.45) (diameter 0) (color 0 0 0 0)
-  )
-  (junction (at 242.57 59.69) (diameter 0) (color 0 0 0 0)
-  )
   (junction (at 113.03 128.27) (diameter 0) (color 0 0 0 0)
   )
-  (junction (at 213.36 120.65) (diameter 0) (color 0 0 0 0)
-  )
-  (junction (at 219.71 59.69) (diameter 0) (color 0 0 0 0)
-  )
-  (junction (at 101.6 157.48) (diameter 0) (color 0 0 0 0)
-  )
-  (junction (at 39.37 186.69) (diameter 0) (color 0 0 0 0)
-  )
-  (junction (at 67.31 67.31) (diameter 0) (color 0 0 0 0)
-  )
-  (junction (at 201.93 120.65) (diameter 0) (color 0 0 0 0)
-  )
-  (junction (at 52.07 186.69) (diameter 0) (color 0 0 0 0)
-  )
-  (junction (at 52.07 179.07) (diameter 0) (color 0 0 0 0)
-  )
-  (junction (at 50.8 165.1) (diameter 0) (color 0 0 0 0)
-  )
-  (junction (at 25.4 157.48) (diameter 0) (color 0 0 0 0)
-  )
-  (junction (at 25.4 165.1) (diameter 0) (color 0 0 0 0)
-  )
-  (junction (at 88.9 165.1) (diameter 0) (color 0 0 0 0)
-  )
-  (junction (at 90.17 124.46) (diameter 0) (color 0 0 0 0)
-  )
-  (junction (at 25.4 179.07) (diameter 0) (color 0 0 0 0)
-  )
-  (junction (at 101.6 165.1) (diameter 0) (color 0 0 0 0)
-  )
-  (junction (at 50.8 109.22) (diameter 0) (color 0 0 0 0)
-  )
   (junction (at 219.71 44.45) (diameter 0) (color 0 0 0 0)
   )
@@
     (stroke (width 0) (type default))
   )
+  (wire (pts (xy 113.03 63.5) (xy 116.84 63.5))
+    (stroke (width 0) (type default))
+  )
   (wire (pts (xy 50.8 44.45) (xy 67.31 44.45))
     (stroke (width 0) (type default))
@@
     (stroke (width 0) (type default))
   )
+  (wire (pts (xy 113.03 128.27) (xy 116.84 128.27))
+    (stroke (width 0) (type default))
+  )
   (polyline (pts (xy 234.95 113.03) (xy 234.95 134.62))
     (stroke (width 0) (type default))
@@
     (stroke (width 0) (type default))
   )
-  (wire (pts (xy 113.03 63.5) (xy 116.84 63.5))
-    (stroke (width 0) (type default))
-  )
   (wire (pts (xy 229.87 33.02) (xy 219.71 33.02))
     (stroke (width 0) (type default))
@@
   )
   (wire (pts (xy 101.6 165.1) (xy 114.3 165.1))
-    (stroke (width 0) (type default))
-  )
-  (wire (pts (xy 113.03 128.27) (xy 116.84 128.27))
     (stroke (width 0) (type default))
   )
@@
     (effects (font (size 1.27 1.27)) (justify left))
   )
-  (hierarchical_label "OP3O" (shape output) (at 116.84 128.27 0) (fields_autoplaced)
+  (hierarchical_label "OP3O" (shape output) (at 116.84 63.5 0) (fields_autoplaced)
     (effects (font (size 1.27 1.27)) (justify left))
   )
@@
     (effects (font (size 1.27 1.27)) (justify left))
   )
-  (hierarchical_label "OP1O" (shape output) (at 116.84 63.5 0) (fields_autoplaced)
+  (hierarchical_label "OP1O" (shape output) (at 116.84 128.27 0) (fields_autoplaced)
     (effects (font (size 1.27 1.27)) (justify left))
   )
