File: hardware/moco-pg4_2/moco-pg4_2.kicad_pcb (KiCad board)
At the start: 6 copper layers, 32 x 32 mm, 100 parts, among them J1 Debug, J2 CAN, J3 V+, J4 V-, J5 A, J6 B, J7 C, J8 CAN, Q1 CSD88584Q5DC, Q2 CSD88584Q5DC, Q7 CSD88584Q5DC, SW1 RESET, U1 STSPIN32G4, U2 TCAN337, U3 MA702, Y1 24MHz

Commit message: Routed moco-SC1 rev1
Parts:
- added J3: V+, moco:wire_2.2mm_rectagnel, F.Cu at (119.6, 42.9)
- added J4: V-, moco:wire_2.2mm, F.Cu at (115.0, 42.8)
Changed lines of the file:
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@@
     )
   )
+  (footprint "moco:wire_2.2mm_rectagnel" (layer "F.Cu")
+    (at 119.614181 42.9 90)
+    (property "Sheetfile" "moco-pg4_2.kicad_sch")
+    (property "Sheetname" "")
+    (property "ki_description" "Generic connector, single row, 01x01, script generated (kicad-library-utils/schlib/autogen/connector/)")
+    (property "ki_keywords" "connector")
+    (attr through_hole)
+    (fp_text reference "J3" (at 0 0 90 unlocked) (layer "F.SilkS") hide
+        (effects (font (size 1 1) (thickness 0.1)))
+    )
+    (fp_text value "V+" (at 0 3 90 unlocked) (layer "F.Fab") hide
+        (effects (font (size 1 1) (thickness 0.15)))
+    )
+    (fp_rect (start -2 -2) (end 2 2)
+      (stroke (width 0.05) (type default)) (fill none) (layer "F.CrtYd"))
+    (pad "1" thru_hole circle (at -1.385819 -0.574025 315) (size 0.7 0.7) (drill 0.4) (layers "*.Cu" "*.Mask")
+      (pinfunction "Pin_1") (pintype "passive"))
+    (pad "1" thru_hole circle (at -1.385819 0.574025 315) (size 0.7 0.7) (drill 0.4) (layers "*.Cu" "*.Mask")
+      (pinfunction "Pin_1") (pintype "passive"))
+    (pad "1" thru_hole circle (at -0.574025 -1.385819 315) (size 0.7 0.7) (drill 0.4) (layers "*.Cu" "*.Mask")
+      (pinfunction "Pin_1") (pintype "passive"))
+    (pad "1" thru_hole circle (at -0.574025 1.385819 315) (size 0.7 0.7) (drill 0.4) (layers "*.Cu" "*.Mask")
+      (pinfunction "Pin_1") (pintype "passive"))
+    (pad "1" thru_hole roundrect (at 0 0 90) (size 3.7 3.7) (drill 2.2) (layers "*.Cu" "*.Mask") (roundrect_rratio 0.15)
+      (pinfunction "Pin_1") (pintype "passive"))
+    (pad "1" thru_hole circle (at 0.574025 -1.385819 315) (size 0.7 0.7) (drill 0.4) (layers "*.Cu" "*.Mask")
+      (pinfunction "Pin_1") (pintype "passive"))
+    (pad "1" thru_hole circle (at 0.574025 1.385819 315) (size 0.7 0.7) (drill 0.4) (layers "*.Cu" "*.Mask")
+      (pinfunction "Pin_1") (pintype "passive"))
+    (pad "1" thru_hole circle (at 1.385819 -0.574025 315) (size 0.7 0.7) (drill 0.4) (layers "*.Cu" "*.Mask")
+      (pinfunction "Pin_1") (pintype "passive"))
+    (pad "1" thru_hole circle (at 1.385819 0.574025 315) (size 0.7 0.7) (drill 0.4) (layers "*.Cu" "*.Mask")
+      (pinfunction "Pin_1") (pintype "passive"))
+  )
   (footprint "Resistor_SMD:R_0402_1005Metric" (layer "F.Cu")
     (at 113.2 73.458335)
@@
     )
   )
+  (footprint "moco:wire_2.2mm" (layer "F.Cu")
+    (at 115 42.814181)
+    (property "Sheetfile" "moco-pg4_2.kicad_sch")
+    (property "Sheetname" "")
+    (property "ki_description" "Generic connector, single row, 01x01, script generated (kicad-library-utils/schlib/autogen/connector/)")
+    (property "ki_keywords" "connector")
+    (attr through_hole)
+    (fp_text reference "J4" (at 0 0 unlocked) (layer "F.SilkS") hide
+        (effects (font (size 1 1) (thickness 0.1)))
+    )
+    (fp_text value "V-" (at 0 3 unlocked) (layer "F.Fab") hide
+        (effects (font (size 1 1) (thickness 0.15)))
+    )
+    (fp_circle (center 0 0) (end 2 0)
+      (stroke (width 0.05) (type default)) (fill none) (layer "F.CrtYd"))
+    (pad "1" thru_hole circle (at -1.385819 -0.574025 225) (size 0.7 0.7) (drill 0.4) (layers "*.Cu" "*.Mask")
+      (pinfunction "Pin_1") (pintype "passive"))
+    (pad "1" thru_hole circle (at -1.385819 0.574025 225) (size 0.7 0.7) (drill 0.4) (layers "*.Cu" "*.Mask")
+      (pinfunction "Pin_1") (pintype "passive"))
+    (pad "1" thru_hole circle (at -0.574025 -1.385819 225) (size 0.7 0.7) (drill 0.4) (layers "*.Cu" "*.Mask")
+      (pinfunction "Pin_1") (pintype "passive"))
+    (pad "1" thru_hole circle (at -0.574025 1.385819 225) (size 0.7 0.7) (drill 0.4) (layers "*.Cu" "*.Mask")
+      (pinfunction "Pin_1") (pintype "passive"))
+    (pad "1" thru_hole circle (at 0 0) (size 3.7 3.7) (drill 2.2) (layers "*.Cu" "*.Mask")
+      (pinfunction "Pin_1") (pintype "passive"))
+    (pad "1" thru_hole circle (at 0.574025 -1.385819 225) (size 0.7 0.7) (drill 0.4) (layers "*.Cu" "*.Mask")
+      (pinfunction "Pin_1") (pintype "passive"))
+    (pad "1" thru_hole circle (at 0.574025 1.385819 225) (size 0.7 0.7) (drill 0.4) (layers "*.Cu" "*.Mask")
+      (pinfunction "Pin_1") (pintype "passive"))
+    (pad "1" thru_hole circle (at 1.385819 -0.574025 225) (size 0.7 0.7) (drill 0.4) (layers "*.Cu" "*.Mask")
+      (pinfunction "Pin_1") (pintype "passive"))
+    (pad "1" thru_hole circle (at 1.385819 0.574025 225) (size 0.7 0.7) (drill 0.4) (layers "*.Cu" "*.Mask")
+      (pinfunction "Pin_1") (pintype "passive"))
+  )
   (footprint "Capacitor_SMD:C_0402_1005Metric" (layer "F.Cu")
     (at 97.27 59.762499)
@@
   (segment (start 101.275 72.589302) (end 101.275 62.9068) (width 0.2) (layer "B.Cu") (net 50))
   (via (at 104.507501 74.76) (size 0.7) (drill 0.3) (layers "F.Cu" "B.Cu") (net 51))
-  (segment (start 110.2 68.07468) (end 110.2 66.4) (width 0.2) (layer "B.Cu") (net 51))
-  (segment (start 104.507501 73.767179) (end 110.2 68.07468) (width 0.2) (layer "B.Cu") (net 51))
+  (segment (start 104.507501 74.76) (end 104.507501 73.767179) (width 0.2) (layer "B.Cu") (net 51))
+  (segment (start 110.078232 68.196448) (end 110.078232 66.521768) (width 0.2) (layer "B.Cu") (net 51))
+  (segment (start 115.965635 65.483835) (end 117 66.5182) (width 0.2) (layer "B.Cu") (net 51))
   (segment (start 116.541665 67.458335) (end 115.7 67.458335) (width 0.2) (layer "B.Cu") (net 51))
-  (segment (start 117 66.5182) (end 117 67) (width 0.2) (layer "B.Cu") (net 51))
+  (segment (start 110.078232 66.521768) (end 111.116165 65.483835) (width 0.2) (layer "B.Cu") (net 51))
   (segment (start 111.116165 65.483835) (end 115.965635 65.483835) (width 0.2) (layer "B.Cu") (net 51))
-  (segment (start 115.965635 65.483835) (end 117 66.5182) (width 0.2) (layer "B.Cu") (net 51))
-  (segment (start 104.507501 74.76) (end 104.507501 73.767179) (width 0.2) (layer "B.Cu") (net 51))
   (segment (start 117 67) (end 116.541665 67.458335) (width 0.2) (layer "B.Cu") (net 51))
-  (segment (start 110.2 66.4) (end 111.116165 65.483835) (width 0.2) (layer "B.Cu") (net 51))
+  (segment (start 117 66.5182) (end 117 67) (width 0.2) (layer "B.Cu") (net 51))
+  (segment (start 104.507501 73.767179) (end 110.078232 68.196448) (width 0.2) (layer "B.Cu") (net 51))
   (via (at 114 70.2) (size 0.7) (drill 0.3) (layers "F.Cu" "B.Cu") (free) (net 52))
   (segment (start 104.825144 75.442357) (end 105.507501 74.76) (width 0.2) (layer "F.Cu") (net 54))
