File: hardware/moco-pg4_3/power_stage.kicad_sch (KiCad schematic)
At the start: 57 parts, among them Q1 CSD88584Q5DC, Q2 CSD88584Q5DC, Q7 CSD88584Q5DC

Commit message: Routed moco-SC1 rev1
Parts:
- added C16, C20, C24: 4.7nF/50V, Capacitor_SMD:C_0402_1005Metric, symbol Device:C_Small
- added C25: 22uF/50V, Capacitor_SMD:CP_Elec_5x5.8, symbol Device:C_Polarized
- added C? (x9): 10uF/50V, Capacitor_SMD:C_0805_2012Metric, symbol Device:C
- added R? (x3): 2.2R/125mW, Resistor_SMD:R_0805_2012Metric, symbol Device:R_Small
- C? (x3): value 100nF -> 1nF; LCSC C5378 -> C1523; MFR. Part# CL21B224KBFNNNE -> 0402B102K500NT
- J? (x3): footprint moco:wire_2.2mm_rectagnel -> moco:wire_rectagnel_3.7mm_D1.5mm
- Q1: renamed from Q2; LCSC (none) -> C2683056; MFR. Part# (none) -> CSD88584Q5DC
- Q2: renamed from Q1; LCSC (none) -> C2683056; MFR. Part# (none) -> CSD88584Q5DC
- Q3: renamed from Q7; LCSC (none) -> C2683056; MFR. Part# (none) -> CSD88584Q5DC
Connections:
- net GNDPWR: now also C25.2, C?.2, C?.2, C?.2, C?.2, C?.2, C?.2, C?.2, C?.2, C?.2, R?.2, R?.2, R?.2
- net OUTA: now also Q1.10 (VSW), Q1.11 (VSW), Q1.3 (VSW), Q1.4 (VSW), Q1.5 (VSW), Q1.6 (VSW), Q1.7 (VSW), Q1.8 (VSW), Q1.9 (VSW), C16.1; no longer Q3.10 (VSW), Q3.11 (VSW), Q3.3 (VSW), Q3.4 (VSW), Q3.5 (VSW), Q3.6 (VSW), Q3.7 (VSW), Q3.8 (VSW), Q3.9 (VSW)
- net OUTB: now also C20.1
- net OUTC: now also Q3.10 (VSW), Q3.11 (VSW), Q3.3 (VSW), Q3.4 (VSW), Q3.5 (VSW), Q3.6 (VSW), Q3.7 (VSW), Q3.8 (VSW), Q3.9 (VSW), C24.1; no longer Q1.10 (VSW), Q1.11 (VSW), Q1.3 (VSW), Q1.4 (VSW), Q1.5 (VSW), Q1.6 (VSW), Q1.7 (VSW), Q1.8 (VSW), Q1.9 (VSW)
- net RSA+: now also NT?.1; no longer NT?.1
- net RSA-: now also NT?.1; no longer NT?.1
- net RSC+: now also NT?.1; no longer NT?.1
- net RSC-: now also NT?.1; no longer NT?.1
- net S2A: now also NT?.2, Q1.12 (PGND), Q1.13 (PGND), Q1.14 (PGND), Q1.15 (PGND), Q1.16 (PGND), Q1.17 (PGND), Q1.18 (PGND), Q1.19 (PGND), Q1.20 (PGND), R?.1; no longer NT?.2, Q3.12 (PGND), Q3.13 (PGND), Q3.14 (PGND), Q3.15 (PGND), Q3.16 (PGND), Q3.17 (PGND), Q3.18 (PGND), Q3.19 (PGND), Q3.20 (PGND), R?.1
- net S2C: now also NT?.2, Q3.12 (PGND), Q3.13 (PGND), Q3.14 (PGND), Q3.15 (PGND), Q3.16 (PGND), Q3.17 (PGND), Q3.18 (PGND), Q3.19 (PGND), Q3.20 (PGND), R?.1; no longer NT?.2, Q1.12 (PGND), Q1.13 (PGND), Q1.14 (PGND), Q1.15 (PGND), Q1.16 (PGND), Q1.17 (PGND), Q1.18 (PGND), Q1.19 (PGND), Q1.20 (PGND), R?.1
- net VBUS: now also C25.1, C?.1, C?.1, C?.1, C?.1, C?.1, C?.1, C?.1, C?.1, C?.1
- net at R?.1: now also U?.29 (GLS1); no longer U?.31 (GLS3)
- net at C?.1, U?.42 (OUT1): now also Q1.2 (SH); no longer Q3.2 (SH)
- net at R?.1: now also U?.31 (GLS3); no longer U?.29 (GLS1)
- net at R?.1: now also U?.37 (GHS3); no longer U?.43 (GHS1)
- net at R?.1: now also U?.43 (GHS1); no longer U?.37 (GHS3)
- net at C?.1, U?.36 (OUT3): now also Q3.2 (SH); no longer Q1.2 (SH)
- new net: C20.2, R?.1
- new net: C16.2, R?.1
- new net: C24.2, R?.1
Other:
- note added: "Gain_{max} = V_{DD}/(2*I_{max}*R_{S}) I_{max} = 12A, Gain_{max} = 6.875 Gain = R_{B}/R_{A} ≈ 6.74 Refer to ST AN5397"
- note added: "RC snubber"
- note added: "STM32 internal Op-Amp"
- note removed: "STM32G432 internal OP-Amp"
- moved on the sheet: C?, Q1, Q3, R?
