File: hardware/moco-sc1/power_stage.kicad_sch (KiCad schematic)
At the start: 73 parts, among them Q1 CSD88584Q5DC, Q2 CSD88584Q5DC, Q3 CSD88584Q5DC

Commit message: Update parts
Parts:
- C? (x18): Alt. (none) -> CL21B106KAYQNNE
- R? (x3): LCSC C840620 -> (none); MFR. Part# CRA2512-FZ-R020ELF -> MSMA2512R0200FGM
