File: hardware/moco-sc1/rotary_sensor.kicad_sch (KiCad schematic)
At the start: 2 parts

Commit message: Update parts
Parts:
- U?: Alt. (none) -> MA730
Changed lines of the file:
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@@
         )
       )
-      (project "moco-pg4_2"
+      (project "moco-sc1"
         (path "/cac36919-bfa9-4a4d-8aba-473f26666d98/6c2b3782-0b5b-4b71-bad7-2198715f7b1c"
           (reference "#PWR054") (unit 1)
@@
         )
       )
-      (project "moco-pg4_2"
+      (project "moco-sc1"
         (path "/cac36919-bfa9-4a4d-8aba-473f26666d98/6c2b3782-0b5b-4b71-bad7-2198715f7b1c"
           (reference "C46") (unit 1)
@@
     )
     (property "MFR. Part#" "MA702GQ-Z " (at 90.17 68.58 0)
+      (effects (font (size 1.27 1.27)) hide)
+    )
+    (property "Alt." "MA730" (at 90.17 68.58 0)
       (effects (font (size 1.27 1.27)) hide)
     )
@@
         )
       )
-      (project "moco-pg4_2"
+      (project "moco-sc1"
         (path "/cac36919-bfa9-4a4d-8aba-473f26666d98/6c2b3782-0b5b-4b71-bad7-2198715f7b1c"
           (reference "U3") (unit 1)
@@
         )
       )
-      (project "moco-pg4_2"
+      (project "moco-sc1"
         (path "/cac36919-bfa9-4a4d-8aba-473f26666d98/6c2b3782-0b5b-4b71-bad7-2198715f7b1c"
           (reference "#PWR053") (unit 1)
@@
         )
       )
-      (project "moco-pg4_2"
+      (project "moco-sc1"
         (path "/cac36919-bfa9-4a4d-8aba-473f26666d98/6c2b3782-0b5b-4b71-bad7-2198715f7b1c"
           (reference "#PWR052") (unit 1)
