File: hardware/moco-sc1/moco-sc1.kicad_sch (KiCad schematic)
At the start: 45 parts, among them U1 STSPIN32G4, U2 TCAN337, Y1 16MHz

Commit message: Update parts
Parts:
- C?: Alt. (none) -> CL21B106KAYQNNE
- D?: value STPS0560Z -> MBR180S1; Alt. (none) -> STPS0560Z; LCSC C99285 -> C526660; MFR. Part# STPS0560Z -> MBR180S1-7
- J? (x2): footprint Connector_JST:JST_SH_SM03B-SRSS-TB_1x03-1MP_P1.00mm_Horizontal -> Connector_JST:JST_GH_SM03B-GHS-TB_1x03-1MP_P1.25mm_Horizontal; LCSC C160403 -> (none); MFR. Part# SM03B-SRSS-TB(LF)(SN) -> (none)
- L?: footprint Inductor_SMD:L_Sunlord_SWPA3012S -> Inductor_SMD:L_Neosid_SMS-ME3015; Alt. (none) -> SRN3015C-180M
- U2: footprint Package_TO_SOT_SMD:SOT-23-8 -> Package_SO:SOIC-8_3.9x4.9mm_P1.27mm; Alt. (none) -> TCAN33x; LCSC C130129 -> C73651; MFR. Part# TCAN337DCNR -> TCAN332DR
