File: hardware/moco-sc2/moco-sc2.kicad_pcb (KiCad board)
At the start: 4 copper layers, 40 x 40 mm, 118 parts, among them J1 Debug, J2 CAN, J3 CAN, J4 V+, J5 V-, J6 A, J7 B, J8 C, Q1 CSD88584Q5DC, Q2 CSD88584Q5DC, Q3 CSD88584Q5DC, SW1 RESET, U1 STSPIN32G4, U2 TCAN337, U3 MA702, Y1 16MHz

Commit message: Update SC2
Parts:
- removed C16, C20, C24: 4.7nF/50V, Capacitor_SMD:C_0402_1005Metric
- removed C27: 22uF/50V, Capacitor_SMD:CP_Elec_5x5.8
- removed R18, R27, R9: 2.2R/125mW, Resistor_SMD:R_0805_2012Metric
- C40, C41, C42, C43, C44, C45: moved to F.Cu
- Q1, Q2, Q3: value CSD88584Q5DC -> SiZF906BDT; footprint moco:VSON-CLIP-22_5x6mm (DMM0022A)_Alt1 -> moco:PowerPAIR_6x5F
- moved kibuzzard-64C58EFF 40.9 mm to (72.0, 49.5)
- moved J5 35.5 mm to (116.0, 42.5)
- moved J4 35.3 mm to (120.8, 42.4)
- moved C31 17.1 mm to (135.6, 71.0)
- moved C32 17.1 mm to (135.6, 69.5)
- moved C33 17.1 mm to (135.6, 68.0)
- moved C37 17.1 mm to (135.6, 61.0)
- moved C38 17.1 mm to (135.6, 59.5)
- moved C39 17.1 mm to (135.6, 58.0)
- moved C23 17.1 mm to (139.1, 64.5)
- moved C28 17.1 mm to (139.1, 71.0)
- moved C29 17.1 mm to (139.1, 69.5)
- moved C30 17.1 mm to (139.1, 68.0)
- moved C34 17.1 mm to (139.1, 61.0)
- moved C35 17.1 mm to (139.1, 59.5)
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Connections:
- Q1 pad 10: /Power Stage/OUTA -> VBUS
- Q1 pad 3: /Power Stage/OUTA -> VBUS
- Q1 pad 4: /Power Stage/OUTA -> VBUS
- Q1 pad 8: /Power Stage/OUTA -> Net-(Q1-G2)
- Q1 pad 9: /Power Stage/OUTA -> /Power Stage/S2A
- Q2 pad 10: /Power Stage/OUTB -> VBUS
- Q2 pad 3: /Power Stage/OUTB -> VBUS
- Q2 pad 4: /Power Stage/OUTB -> VBUS
- Q2 pad 8: /Power Stage/OUTB -> Net-(Q2-G2)
- Q2 pad 9: /Power Stage/OUTB -> /Power Stage/S2B
- Q3 pad 10: /Power Stage/OUTC -> VBUS
- Q3 pad 3: /Power Stage/OUTC -> VBUS
- Q3 pad 4: /Power Stage/OUTC -> VBUS
- Q3 pad 8: /Power Stage/OUTC -> Net-(Q3-G2)
- Q3 pad 9: /Power Stage/OUTC -> /Power Stage/S2C
- R11 pad 2: Net-(Q1-GL) -> Net-(Q1-G2)
- R20 pad 2: Net-(Q2-GL) -> Net-(Q2-G2)
- R29 pad 2: Net-(Q3-GL) -> Net-(Q3-G2)
Routing:
- net +3.3V: track 95.2 -> 0.00 mm, vias 9 -> 0
- net VBUS: track 85.1 -> 0.00 mm, vias 12 -> 0
- net GND: track 54.3 -> 0.00 mm, vias 108 -> 0
- net /Power Stage/RSA+: track 46.8 -> 0.00 mm, vias 1 -> 0
- net /Power Stage/RSA-: track 44.7 -> 0.00 mm, vias 1 -> 0
- net /Power Stage/RSB-: track 43.7 -> 0.00 mm, vias 1 -> 0
- net /Power Stage/RSB+: track 37.9 -> 0.00 mm, vias 1 -> 0
- net /USER_LED: track 32.9 -> 0.00 mm, vias 2 -> 0
- net /Power Stage/RSC-: track 29.2 -> 0.00 mm, vias 1 -> 0
- net /Power Stage/RSC+: track 28.6 -> 0.00 mm, vias 1 -> 0
- net Net-(U1C-GLS1): track 27.5 -> 0.00 mm, vias 2 -> 0
- net /SWCLK: track 24.9 -> 0.00 mm, vias 1 -> 0
- net /SWO: track 24.1 -> 0.00 mm, vias 1 -> 0
- net /USART_RX: track 24.0 -> 0.00 mm
- net VCC: track 23.9 -> 0.00 mm, vias 2 -> 0
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- removed copper zone on F.Cu, net /Power Stage/OUTA
- removed copper zone on F.Cu, net /Power Stage/OUTB
- removed copper zone on F.Cu, net /Power Stage/OUTC
- removed copper zone on B.Cu, net /Power Stage/S2A
- removed copper zone on F.Cu, net /Power Stage/S2A
- removed copper zone on B.Cu, net /Power Stage/S2B
- removed copper zone on F.Cu, net /Power Stage/S2B
- removed copper zone on B.Cu, net /Power Stage/S2C
- removed copper zone on F.Cu, net /Power Stage/S2C
- removed copper zone on B.Cu, net GND
- removed copper zone on F.Cu, net GND
- removed copper zone on In1.Cu, net GND
- removed copper zone on F.Cu, net Net-(D1-K)
- removed copper zone on B.Cu, net VBUS
- removed copper zone on F.Cu, net VBUS
- removed copper zone on In1.Cu, net VBUS
- removed copper zone on In2.Cu, net VBUS
- removed copper zone on F.Cu, net VCC
