File: hardware/moco-sc2/power_stage.kicad_sch (KiCad schematic)
At the start: 73 parts, among them Q1 CSD88584Q5DC, Q2 CSD88584Q5DC, Q3 CSD88584Q5DC

Commit message: Update SC2
Parts:
- removed C16, C20, C24: 4.7nF/50V, Capacitor_SMD:C_0402_1005Metric, symbol Device:C_Small
- removed C25: 22uF/50V, Capacitor_SMD:CP_Elec_5x5.8, symbol Device:C_Polarized
- removed Q1, Q2, Q3: CSD88584Q5DC, moco:VSON-CLIP-22_5x6mm (DMM0022A)_Alt1, symbol moco:CSD88584Q5DC
- removed R? (x3): 2.2R/125mW, Resistor_SMD:R_0805_2012Metric, symbol Device:R_Small
- added Q1, Q2, Q3: SiZF906BDT, moco:PowerPAIR_6x5F, symbol moco:SiZF906BDT
Connections:
- net OUTA: now also Q1.5 (S1-D2), Q1.6 (S1-D2), Q1.7 (S1-D2)
- net OUTB: now also Q2.5 (S1-D2), Q2.6 (S1-D2), Q2.7 (S1-D2)
- net OUTC: now also Q3.5 (S1-D2), Q3.6 (S1-D2), Q3.7 (S1-D2)
- net S2A: now also Q1.9 (S2)
- net S2B: now also Q2.9 (S2)
- net S2C: now also Q3.9 (S2)
- net VBUS: now also Q1.10 (D1), Q1.3 (D1), Q1.4 (D1), Q2.10 (D1), Q2.3 (D1), Q2.4 (D1), Q3.10 (D1), Q3.3 (D1), Q3.4 (D1)
- net at R?.2: now also Q2.1 (G1)
- net at C?.1, U?.39 (OUT2): now also Q2.2 (G1R)
- net at R?.2: now also Q2.8 (G2)
- net at R?.2: now also Q1.8 (G2)
- net at R?.2: now also Q3.1 (G1)
- net at C?.1, U?.36 (OUT3): now also Q3.2 (G1R)
- net at R?.2: now also Q3.8 (G2)
- net at C?.1, U?.42 (OUT1): now also Q1.2 (G1R)
- net at R?.2: now also Q1.1 (G1)
Other:
- note removed: "RC snubber"
