File: hardware/moco-sp1/moco-sp1.kicad_pcb (KiCad board)
At the start: 4 copper layers, 35 x 35 mm, 89 parts, among them J1 OUT_U, J2 OUT_V, J3 OUT_W, J4 Conn_02x03_Odd_Even, J5 VM+, J6 VM-, J7 CAN, Q1 FDMD8240LET40, Q2 FDMD8240LET40, Q3 FDMD8240LET40, SW1 RESET, U1 STSPIN32F0A, U2 TCAN4550, U3 AS5600, Y1 40MHz

Commit message: Update sp1 pcb
Parts:
- removed C16: 100nF, Capacitor_SMD:C_0402_1005Metric
- removed C20: 10uF/50V, Capacitor_SMD:C_0805_2012Metric
- removed C24: 1nF, Capacitor_SMD:C_0402_1005Metric
- removed D2, D3: TVS, Diode_SMD:D_SOD-323_HandSoldering
- removed D4: LED, LED_SMD:LED_0603_1608Metric
- removed R18: 1.78k, Resistor_SMD:R_0402_1005Metric
- removed R27: 24k, Resistor_SMD:R_0402_1005Metric
- removed R9: 10k, Resistor_SMD:R_0402_1005Metric
- removed RS1, RS2, RS3: 20mΩ/3W, Resistor_SMD:R_2512_6332Metric_Pad1.40x3.35mm_HandSolder
- added C28: 10uF/50V, Capacitor_SMD:C_0805_2012Metric, B.Cu at (118.5, 45.0)
- added C29: 10uF/50V, Capacitor_SMD:C_0805_2012Metric, B.Cu at (118.5, 47.0)
- added C30: 10uF/50V, Capacitor_SMD:C_0805_2012Metric, F.Cu at (118.0, 76.0)
- added C31: 10uF/50V, Capacitor_SMD:C_0805_2012Metric, F.Cu at (118.0, 74.0)
- added C32: 10uF/50V, Capacitor_SMD:C_0805_2012Metric, F.Cu at (118.0, 72.0)
- added C33: 10uF/50V, Capacitor_SMD:C_0805_2012Metric, F.Cu at (118.0, 70.0)
- added C34: 10uF/50V, Capacitor_SMD:C_0805_2012Metric, B.Cu at (118.5, 43.0)
- added C35: 10uF/50V, Capacitor_SMD:C_0805_2012Metric, B.Cu at (118.5, 59.5)
- added C36: 10uF/50V, Capacitor_SMD:C_0805_2012Metric, F.Cu at (118.0, 63.5)
- added C37: 10uF/50V, Capacitor_SMD:C_0805_2012Metric, F.Cu at (118.0, 61.5)
- added C38: 10uF/50V, Capacitor_SMD:C_0805_2012Metric, F.Cu at (118.0, 59.5)
- added C39: 10uF/50V, Capacitor_SMD:C_0805_2012Metric, F.Cu at (118.0, 57.5)
- added C40: 10uF/50V, Capacitor_SMD:C_0805_2012Metric, B.Cu at (118.5, 55.5)
- added C41: 10uF/50V, Capacitor_SMD:C_0805_2012Metric, B.Cu at (118.5, 57.5)
- added C42: 10uF/50V, Capacitor_SMD:C_0805_2012Metric, F.Cu at (118.0, 51.0)
- added C43: 10uF/50V, Capacitor_SMD:C_0805_2012Metric, F.Cu at (118.0, 49.0)
- added C44: 10uF/50V, Capacitor_SMD:C_0805_2012Metric, F.Cu at (118.0, 47.0)
- added C45: 10uF/50V, Capacitor_SMD:C_0805_2012Metric, F.Cu at (118.0, 45.0)
- added C46: 1uF, Capacitor_SMD:C_0603_1608Metric_Pad1.08x0.95mm_HandSolder, B.Cu at (107.5, 57.5)
- added H4: MountingHole, MountingHole:MountingHole_3.2mm_M3_ISO14580, F.Cu at (89.0, 81.0)
- added J8: C, moco:wire_rectagnel_3.7mm_D1.5mm, F.Cu at (131.6, 72.6)
- added LD1: Red, LED_SMD:LED_0603_1608Metric, F.Cu at (107.8, 36.8)
- added LD2: Blue, LED_SMD:LED_0603_1608Metric, F.Cu at (106.3, 36.8)
- added Q4: SiDR390DP, Package_SO:PowerPAK_SO-8_Single, F.Cu at (124.0, 50.5)
- added Q5: SiDR390DP, Package_SO:PowerPAK_SO-8_Single, F.Cu at (124.0, 70.0)
- added Q6: SiDR390DP, Package_SO:PowerPAK_SO-8_Single, F.Cu at (124.0, 75.5)
- added R31: 1.78k, Resistor_SMD:R_0402_1005Metric, F.Cu at (101.8, 73.5)
- added R32: 20mΩ/3W, Resistor_SMD:R_2512_6332Metric, B.Cu at (117.0, 75.0)
- added R33: 24k, Resistor_SMD:R_0402_1005Metric, F.Cu at (101.3, 71.0)
- added R34: 1.78k, Resistor_SMD:R_0402_1005Metric, F.Cu at (102.8, 73.5)
- added R35: 12k, Resistor_SMD:R_0402_1005Metric, F.Cu at (103.3, 72.0)
- added SB1: SolderJumper_2_Open, Jumper:SolderJumper-2_P1.3mm_Open_RoundedPad1.0x1.5mm, B.Cu at (66.0, 72.0)
- added TP1: CANH, TestPoint:TestPoint_Pad_D1.0mm, B.Cu at (59.2, 62.8)
- added TP2: CANL, TestPoint:TestPoint_Pad_D1.0mm, B.Cu at (59.2, 68.8)
- added TP3: 3.3V, TestPoint:TestPoint_Pad_D1.0mm, B.Cu at (96.3, 61.0)
- added TP4: VCC, TestPoint:TestPoint_Pad_D1.0mm, B.Cu at (95.8, 57.2)
- added TP5: GND, TestPoint:TestPoint_Pad_D1.0mm, B.Cu at (89.5, 70.7)
- added kibuzzard-64C58EFF: G***, kibuzzard-64C58EFF, F.Cu at (103.2, 110.5)
- C1: value 100nF/50V -> 100nF
- C11: value 100nF -> 1uF
- C12: value 300nF -> 100nF
- C13: value 10uF -> 1uF
- C14: value 10nF -> 10uF; footprint Capacitor_SMD:C_0402_1005Metric -> Capacitor_SMD:C_0805_2012Metric
- C15, C8: value 100nF -> 220nF/50V; footprint Capacitor_SMD:C_0402_1005Metric -> Capacitor_SMD:C_0805_2012Metric
- C17: value 4.7nF -> 100nF/50V
- C18: value 100nF -> 1nF; footprint Capacitor_SMD:C_0603_1608Metric_Pad1.08x0.95mm_HandSolder -> Capacitor_SMD:C_0402_1005Metric; moved to F.Cu
- C19: footprint Capacitor_SMD:C_0402_1005Metric -> Capacitor_SMD:C_0805_2012Metric
- C2: value 1nF -> 6.8pF
- C21: value 10uF/50V -> 100nF/50V; footprint Capacitor_SMD:C_0805_2012Metric -> Capacitor_SMD:C_0402_1005Metric
- C22: value 220nF/50V -> 1nF
- C23: value 100nF/50V -> 220nF/50V; footprint Capacitor_SMD:C_0402_1005Metric -> Capacitor_SMD:C_0805_2012Metric
- C25: value 220nF/50V -> 100nF/50V
- C26: value 100nF/50V -> 1nF
- C27: value 1nF -> 22uF/50V; footprint Capacitor_SMD:C_0402_1005Metric -> Capacitor_SMD:CP_Elec_5x5.8
- C3: value 10uF/50V -> 100nF; footprint Capacitor_SMD:C_0805_2012Metric -> Capacitor_SMD:C_0402_1005Metric
- C4: value 10nF -> 6.8pF
- C5: value 12pF -> 10uF/50V; footprint Capacitor_SMD:C_0402_1005Metric -> Capacitor_SMD:C_0805_2012Metric
- C6: value 12pF -> 100nF
- C7: value 47uF -> 10uF; footprint Capacitor_SMD:C_0805_2012Metric -> Capacitor_SMD:C_0402_1005Metric
- C9: value 10uF -> 100nF
- H1, H2, H3: footprint MountingHole:MountingHole_2.2mm_M2_ISO7380 -> MountingHole:MountingHole_3.2mm_M3_ISO14580
- J1: value OUT_U -> Debug; footprint moco:Conn_1x1_3.7_1.5 -> Connector_PinHeader_2.54mm:PinHeader_2x04_P2.54mm_Vertical
- J2: value OUT_V -> CAN; footprint moco:Conn_1x1_3.7_1.5 -> Connector_JST:JST_GH_SM03B-GHS-TB_1x03-1MP_P1.25mm_Horizontal
- J3: value OUT_W -> CAN; footprint moco:Conn_1x1_3.7_1.5 -> Connector_JST:JST_GH_SM03B-GHS-TB_1x03-1MP_P1.25mm_Horizontal; moved to B.Cu
- J4: value Conn_02x03_Odd_Even -> V+; footprint Connector_PinHeader_2.54mm:PinHeader_2x03_P2.54mm_Vertical -> moco:wire_rectagnel_3.7mm_D1.5mm
- J5: value VM+ -> V-; footprint moco:Conn_1x1_3.7_1.5 -> moco:wire_circ_3.7mm_D1.5mm
- J6: value VM- -> A; footprint moco:Conn_1x1_3.7_1.5 -> moco:wire_rectagnel_3.7mm_D1.5mm
- J7: value CAN -> B; footprint Connector_JST:JST_GH_SM03B-GHS-TB_1x03-1MP_P1.25mm_Horizontal -> moco:wire_rectagnel_3.7mm_D1.5mm
- Q1, Q2, Q3: value FDMD8240LET40 -> SiDR390DP; footprint moco:PQFN-12 -> Package_SO:PowerPAK_SO-8_Single
- R1: value 10R -> 120R; footprint Resistor_SMD:R_0402_1005Metric -> Resistor_SMD:R_0402_1005Metric_Pad0.72x0.64mm_HandSolder
- R10, R11: value 60R -> 10R
- R12: value 4.7k -> 24k
- R13: value 4.7k -> 1.78k
- R14: value 10k -> 20mΩ/3W; footprint Resistor_SMD:R_0402_1005Metric -> Resistor_SMD:R_2512_6332Metric; moved to B.Cu
- R15: value 10R -> 24k
- R16, R22: value 10R -> 1.78k
- R17: value 24k -> 12k
- R19: value 1.78k -> 10R
- R2: value 10R -> 10k
- R20: value 24k -> 10R
- R21: value 12k -> 24k
- R23: value 10R -> 20mΩ/3W; footprint Resistor_SMD:R_0402_1005Metric -> Resistor_SMD:R_2512_6332Metric; moved to B.Cu
- R26: value 1.78k -> 12k
- R28: value 12k -> 10R
- R29: value 68k -> 10R
- R3: value 24k -> 100k
- R30: value 10k -> 24k
- R4: value 1.78k -> 22k
- R5: value 1.78k -> 1k
- R6: value 24k -> 10k
- R7: value 12k -> 10k
- SW1: footprint Button_Switch_SMD:SW_SPST_B3U-1000P -> Button_Switch_SMD:SW_SPST_EVQP7C
- U1: value STSPIN32F0A -> STSPIN32G4; footprint moco:VFQFN-48_7x7_EP2.8mm_Pitch0.5mm -> moco:VFQFPN 9X9X1.0 64 PITCH 0.5
- U2: value TCAN4550 -> TCAN337; footprint moco:VQFN-20_3.5_3.5_0.5p -> Package_SO:SOIC-8_3.9x4.9mm_P1.27mm
- U3: value AS5600 -> MA702; footprint Package_SO:SOIC-8_3.9x4.9mm_P1.27mm -> Package_DFN_QFN:QFN-16-1EP_3x3mm_P0.5mm_EP1.75x1.75mm
- Y1: value 40MHz -> 16MHz
- moved J3 103.8 mm to (76.3, 50.8), turned to 90 degrees
- moved H3 101.3 mm to (89.0, 39.0), turned to 90 degrees
- moved J2 93.1 mm to (89.0, 46.5), turned to -90 degrees
- moved C6 81.9 mm to (94.5, 60.0), turned to 0 degrees
- moved U2 81.8 mm to (99.0, 46.5), turned to 180 degrees
- moved Y1 80.1 mm to (91.5, 62.5), turned to 90 degrees
- moved C5 79.9 mm to (101.3, 54.2), turned to 0 degrees
- moved J1 78.7 mm to (103.6, 37.0), turned to -90 degrees
- moved C15 78.3 mm to (118.0, 43.0), turned to 0 degrees
- moved C14 78.2 mm to (94.8, 56.8), turned to 90 degrees
- moved C22 75.6 mm to (99.1, 71.0)
- moved R1 74.7 mm to (94.5, 47.2), turned to 90 degrees
- moved SW1 72.0 mm to (76.3, 70.2), turned to -90 degrees
- moved C27 71.8 mm to (122.5, 38.5), turned to 180 degrees
- moved C25 70.2 mm to (108.6, 68.2), turned to 135 degrees
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Connections:
- C1 pad 1: Net-(U1D-VBOOTU) -> GND
- C1 pad 2: /Power Stage/QO_U -> +3.3V
- C10 pad 1: VM -> GND
- C10 pad 2: GND -> +3.3V
- C11 pad 1: +3.3V -> GND
- C11 pad 2: GND -> +3.3V
- C12 pad 1: Net-(U2-FLTR) -> GND
- C12 pad 2: GND -> +3.3V
- C13 pad 1: /CAN Bus/5V_out -> GND
- C13 pad 2: GND -> +3.3V
- C14 pad 1: Net-(U2-WAKE) -> VCC
- C15 pad 1: +12V -> GND
- C15 pad 2: GND -> VBUS
- C17 pad 1: Net-(C17-Pad1) -> /Power Stage/OUTA
- C17 pad 2: GND -> Net-(U1C-BOOT1)
- C18 pad 1: GND -> /OPAMP1_VOUT
- C18 pad 2: +3.3V -> /OPAMP1_VINM
- C19 pad 1: VM -> GND
- C19 pad 2: GND -> VBUS
- C2 pad 1: /Power Stage/OPA_U -> GND
- C2 pad 2: Net-(U1E-OP3N) -> /OSC_IN
- C21 pad 1: VM -> /Power Stage/OUTB
- C21 pad 2: GND -> Net-(U1D-BOOT2)
- C22 pad 1: VM -> /OPAMP2_VOUT
- C22 pad 2: GND -> /OPAMP2_VINM
- C23 pad 1: Net-(U1C-VBOOTV) -> GND
- C23 pad 2: /Power Stage/QO_V -> VBUS
- C25 pad 1: VM -> /Power Stage/OUTC
- C25 pad 2: GND -> Net-(U1E-BOOT3)
- C26 pad 1: Net-(U1B-VBOOTW) -> /OPAMP3_VOUT
- C26 pad 2: /Power Stage/QO_W -> /OPAMP3_VINM
- C27 pad 1: /Power Stage/OPA_W -> VBUS
- C27 pad 2: Net-(U1G-OP1N) -> GND
- C3 pad 1: VM -> /~{RESET}
- C4 pad 1: /~{RESET} -> GND
- C4 pad 2: GND -> /OSC_OUT
- C5 pad 1: GND -> VBUS
- C5 pad 2: /CAN Bus/OSC_IN -> GND
- C6 pad 1: /CAN Bus/OSC_OUT -> GND
- C6 pad 2: GND -> +3.3V
- C7 pad 1: +3.3V -> GND
- C7 pad 2: GND -> +3.3V
- C8 pad 1: +3.3V -> VBUS
- C9 pad 1: +12V -> GND
- C9 pad 2: GND -> +3.3V
- J1 pad 1: /Power Stage/OUT_U -> +3.3V
- J2 pad 1: /Power Stage/OUT_V -> /CANL
- J3 pad 1: /Power Stage/OUT_W -> /CANL
- J4 pad 1: +3.3V -> VBUS
- J5 pad 1: VM -> GND
- J6 pad 1: GND -> /Power Stage/OUTA
- J7 pad 1: /CAN Bus/CANH -> /Power Stage/OUTB
- L1 pad 1: +3.3V -> Net-(D1-K)
- L1 pad 2: Net-(D1-K) -> VCC
- NT1 pad 1: /Power Stage/QS_U -> /Power Stage/RSA+
- NT1 pad 2: /Power Stage/RS_U+ -> /Power Stage/S2A
- NT2 pad 1: GND -> /Power Stage/RSA-
- NT2 pad 2: /Power Stage/RS_U- -> GND
- NT3 pad 1: /Power Stage/QS_V -> /Power Stage/RSB+
- NT3 pad 2: /Power Stage/RS_V+ -> /Power Stage/S2B
- NT4 pad 1: GND -> /Power Stage/RSB-
- NT4 pad 2: /Power Stage/RS_V- -> GND
- NT5 pad 1: /Power Stage/QS_W -> /Power Stage/RSC+
- NT5 pad 2: /Power Stage/RS_W+ -> /Power Stage/S2C
- NT6 pad 1: GND -> /Power Stage/RSC-
- NT6 pad 2: /Power Stage/RS_W- -> GND
- Q1 pad 1: VM -> /Power Stage/OUTA
- Q1 pad 2: VM -> /Power Stage/OUTA
- Q1 pad 3: VM -> /Power Stage/OUTA
- Q1 pad 4: /Power Stage/QGL_U -> Net-(Q1-G)
- Q1 pad 5: /Power Stage/QS_U -> VBUS
- Q2 pad 1: VM -> /Power Stage/OUTB
- Q2 pad 2: VM -> /Power Stage/OUTB
- Q2 pad 3: VM -> /Power Stage/OUTB
- Q2 pad 4: /Power Stage/QGL_V -> Net-(Q2-G)
- Q2 pad 5: /Power Stage/QS_V -> VBUS
- Q3 pad 1: VM -> /Power Stage/S2B
- Q3 pad 2: VM -> /Power Stage/S2B
- Q3 pad 3: VM -> /Power Stage/S2B
- Q3 pad 4: /Power Stage/QGL_W -> Net-(Q3-G)
- Q3 pad 5: /Power Stage/QS_W -> /Power Stage/OUTB
- R1 pad 1: Net-(U1D-LSU) -> Net-(SB1-B)
- R1 pad 2: /Power Stage/QGL_U -> /CANL
- R10 pad 1: /CAN Bus/CANH -> Net-(U1C-GHS1)
- R10 pad 2: Net-(C17-Pad1) -> Net-(Q1-G)
- R11 pad 1: Net-(C17-Pad1) -> Net-(U1C-GLS1)
- R11 pad 2: /CAN Bus/CANL -> Net-(Q4-G)
- R12 pad 2: /I2C_SCL -> /OPAMP1_VINP
- R13 pad 1: +3.3V -> /Power Stage/RSA+
- R13 pad 2: /I2C_SDA -> /OPAMP1_VINP
- R14 pad 1: Net-(D4-K) -> /Power Stage/S2A
- R15 pad 1: Net-(U1C-HSV) -> /OPAMP1_VINP
- R15 pad 2: /Power Stage/QGH_V -> GND
- R16 pad 1: Net-(U1C-LSV) -> /Power Stage/RSA-
- R16 pad 2: /Power Stage/QGL_V -> /OPAMP1_VINM
- R17 pad 1: +3.3V -> /OPAMP1_VINM
- R17 pad 2: Net-(U1F-OP2P) -> /OPAMP1_VOUT
- R19 pad 1: /Power Stage/RS_U- -> Net-(U1D-GHS2)
- R19 pad 2: Net-(U1F-OP2N) -> Net-(Q2-G)
- R2 pad 1: Net-(U1D-HSU) -> /~{RESET}
- R2 pad 2: /Power Stage/QGH_U -> +3.3V
- R20 pad 1: Net-(U1F-OP2P) -> Net-(U1D-GLS2)
- R20 pad 2: GND -> Net-(Q3-G)
- R21 pad 1: Net-(U1F-OP2N) -> +3.3V
- R21 pad 2: /Power Stage/OPA_V -> /OPAMP2_VINP
- R22 pad 1: Net-(U1B-HSW) -> /Power Stage/RSB+
- R22 pad 2: /Power Stage/QGH_W -> /OPAMP2_VINP
- R23 pad 1: Net-(U1B-LSW) -> /Power Stage/S2B
- R23 pad 2: /Power Stage/QGL_W -> GND
- R24 pad 1: +3.3V -> /OPAMP2_VINP
- R24 pad 2: Net-(U1G-OP1P) -> GND
- R25 pad 1: /Power Stage/RS_W+ -> /Power Stage/RSB-
- R25 pad 2: Net-(U1G-OP1P) -> /OPAMP2_VINM
- R26 pad 1: /Power Stage/RS_W- -> /OPAMP2_VINM
- R26 pad 2: Net-(U1G-OP1N) -> /OPAMP2_VOUT
- R28 pad 1: Net-(U1G-OP1N) -> Net-(U1E-GHS3)
- R28 pad 2: /Power Stage/OPA_W -> Net-(Q5-G)
- R29 pad 1: VM -> Net-(U1E-GLS3)
- R29 pad 2: /VM_sense -> Net-(Q6-G)
- R3 pad 1: +3.3V -> /V_{BUS}_SENSE
- R3 pad 2: Net-(U1E-OP3P) -> VBUS
- R30 pad 1: /VM_sense -> +3.3V
- R30 pad 2: GND -> /OPAMP3_VINP
- R4 pad 1: /Power Stage/RS_V+ -> +3.3V
- R4 pad 2: Net-(U1E-OP3P) -> /SCREF
- R5 pad 1: /Power Stage/RS_V- -> /USER_LED
- R5 pad 2: Net-(U1E-OP3N) -> Net-(LD1-A)
- R6 pad 1: Net-(U1E-OP3P) -> VCC
- R6 pad 2: GND -> Net-(LD2-A)
- R7 pad 1: Net-(U1E-OP3N) -> GND
- R7 pad 2: /Power Stage/OPA_U -> /V_{BUS}_SENSE
- R8 pad 1: +3.3V -> /SCREF
- R8 pad 2: /~{RESET} -> GND
- U1 pad 1: Net-(U1F-OP2P) -> +3.3V
- U1 pad 10: +3.3V -> unconnected-(U1A-PC1-Pad10)
- U1 pad 11: /Current_sense_U -> unconnected-(U1A-PC2-Pad11)
- U1 pad 12: /Current_sense_V -> unconnected-(U1A-PC3-Pad12)
- U1 pad 13: /UART_TX -> /USER_LED
- U1 pad 14: /Current_sense_W -> /OPAMP1_VINP
- U1 pad 15: /User_LED -> /OPAMP1_VOUT
- U1 pad 16: /SPI_SCK -> /OPAMP1_VINM
- U1 pad 17: /SPI_MISO -> /V_{BUS}_SENSE
- U1 pad 18: /SPI_MOSI -> unconnected-(U1A-PA5-Pad18)
- U1 pad 19: /VM_sense -> /OPAMP2_VOUT
- U1 pad 2: Net-(U1F-OP2N) -> +3.3V
- U1 pad 20: GND -> /OPAMP2_VINP
- U1 pad 21: /Power Stage/OPA_W -> unconnected-(U1A-PC4-Pad21)
- U1 pad 22: Net-(U1G-OP1N) -> /OPAMP2_VINM
- U1 pad 23: Net-(U1G-OP1P) -> /OPAMP3_VINP
- U1 pad 24: /OC_COMP -> /OPAMP3_VOUT
- U1 pad 25: Net-(U1B-HSW) -> /OPAMP3_VINM
- U1 pad 26: /Power Stage/QO_W -> +3.3V
- U1 pad 27: Net-(U1B-VBOOTW) -> +3.3V
- U1 pad 28: Net-(U1B-LSW) -> unconnected-(U1A-PB10-Pad28)
- U1 pad 29: Net-(U1C-HSV) -> Net-(U1C-GLS1)
- U1 pad 3: /Power Stage/OPA_V -> unconnected-(U1A-PC13-Pad3)
- U1 pad 30: /Power Stage/QO_V -> Net-(U1D-GLS2)
- U1 pad 31: Net-(U1C-VBOOTV) -> Net-(U1E-GLS3)
- U1 pad 32: Net-(U1C-LSV) -> GND
- U1 pad 33: Net-(U1D-HSU) -> unconnected-(U1A-NC-Pad33)
- U1 pad 34: /Power Stage/QO_U -> unconnected-(U1A-NC-Pad34)
- U1 pad 35: Net-(U1D-VBOOTU) -> Net-(U1E-BOOT3)
- U1 pad 36: Net-(U1D-LSU) -> /Power Stage/OUTC
- U1 pad 37: /SWD -> Net-(U1E-GHS3)
- U1 pad 38: /SWC -> Net-(U1D-BOOT2)
- U1 pad 39: /UART_RX -> /Power Stage/OUTB
- U1 pad 4: /SPI_IRQ -> unconnected-(U1A-PC14-Pad4)
- U1 pad 40: /I2C_SCL -> Net-(U1D-GHS2)
- U1 pad 41: /I2C_SDA -> Net-(U1C-BOOT1)
- U1 pad 42: /BOOT0 -> /Power Stage/OUTA
- U1 pad 43: unconnected-(U1A-RESERVED-Pad43) -> Net-(U1C-GHS1)
- U1 pad 44: GND -> unconnected-(U1A-PA8-Pad44)
- U1 pad 45: Net-(U1E-OP3P) -> /USART_TX
- U1 pad 46: Net-(U1E-OP3N) -> /USART_RX
- U1 pad 47: /Power Stage/OPA_U -> /CAN_RX
- U1 pad 48: +3.3V -> /CAN_TX
- U1 pad 49: GND -> /SWDIO
- U1 pad 5: /SPI_~{CS} -> unconnected-(U1A-PC15-Pad5)
- U1 pad 6: +12V -> /OSC_IN
- U1 pad 7: /~{RESET} -> /OSC_OUT
- U1 pad 8: VM -> /~{RESET}
- U1 pad 9: Net-(D1-K) -> unconnected-(U1A-PC0-Pad9)
- U2 pad 1: /CAN Bus/OSC_IN -> /CAN_TX
- U2 pad 2: /CAN Bus/~{WKRQ} -> GND
- U2 pad 3: unconnected-(U2-GPO1-Pad3) -> +3.3V
- U2 pad 4: /SPI_SCK -> /CAN_RX
- U2 pad 5: /SPI_MOSI -> unconnected-(U2-FAULT-Pad5)
- U2 pad 6: /SPI_MISO -> /CANL
- U2 pad 7: /SPI_~{CS} -> /CANH
- U2 pad 8: /SPI_IRQ -> unconnected-(U2-S-Pad8)
- U3 pad 1: +3.3V -> unconnected-(U3-SSD-Pad1)
- U3 pad 2: +3.3V -> /Rotary Sensor/A
- U3 pad 3: unconnected-(U3-OUT-Pad3) -> /Rotary Sensor/Z
- U3 pad 4: GND -> /SPI_MOSI
- U3 pad 5: unconnected-(U3-PGO-Pad5) -> /SPI_~{CS}_RS
- U3 pad 6: /I2C_SDA -> /Rotary Sensor/B
- U3 pad 7: /I2C_SCL -> /SPI_MISO
- U3 pad 8: unconnected-(U3-DIR-Pad8) -> GND
- Y1 pad 1: /CAN Bus/OSC_OUT -> /OSC_OUT
- Y1 pad 3: /CAN Bus/OSC_IN -> /OSC_IN
Routing:
- net VM: vias 6 -> 0
Other:
- board size 35 x 35 mm -> 50 x 50 mm
- board text added: "+10~35V"
- board text added: "3.3V"
- board text added: "G"
- board text added: "GND PWR"
- board text added: "H"
- board text added: "L"
- board text added: "SIGNAL"
- board text added: "v${REVISION}"
