File: hardware/moco-sp1/moco-sp1.kicad_sch (KiCad schematic)
At the start: 25 parts, among them J4 Conn_02x03_Odd_Even, J5 VM+, J6 VM-, SW1 RESET, U1 STSPIN32F0A

Commit message: Update sp1 pcb
Parts:
- removed C10, C11, C8: 100nF, Capacitor_SMD:C_0402_1005Metric, symbol Device:C
- removed C3: 10uF/50V, Capacitor_SMD:C_0805_2012Metric, symbol Device:C
- removed C4: 10nF, Capacitor_SMD:C_0402_1005Metric, symbol Device:C
- removed C7: 47uF, Capacitor_SMD:C_0805_2012Metric, symbol Device:C
- removed C9: 10uF, Capacitor_SMD:C_0402_1005Metric, symbol Device:C
- removed D1: MBR180S1, Diode_SMD:D_SOD-123F, symbol Diode:1N6857UR
- removed D4: LED, LED_SMD:LED_0603_1608Metric, symbol Device:LED
- removed H1, H2, H3: MountingHole, MountingHole:MountingHole_2.2mm_M2_ISO7380, symbol Mechanical:MountingHole
- removed J4: Conn_02x03_Odd_Even, Connector_PinHeader_2.54mm:PinHeader_2x03_P2.54mm_Vertical, symbol Connector_Generic:Conn_02x03_Odd_Even
- removed J5: VM+, moco:Conn_1x1_3.7_1.5, symbol Connector_Generic:Conn_01x01
- removed J6: VM-, moco:Conn_1x1_3.7_1.5, symbol Connector_Generic:Conn_01x01
- removed L1: 18uH, Inductor_SMD:L_Neosid_SMS-ME3015, symbol Device:L
- removed R12, R13: 4.7k, Resistor_SMD:R_0402_1005Metric, symbol Device:R
- removed R14, R30, R9: 10k, Resistor_SMD:R_0402_1005Metric, symbol Device:R
- removed R29: 68k, Resistor_SMD:R_0402_1005Metric, symbol Device:R
- removed SW1: RESET, Button_Switch_SMD:SW_SPST_B3U-1000P, symbol Switch:SW_Push
- removed U1: STSPIN32F0A, moco:VFQFN-48_7x7_EP2.8mm_Pitch0.5mm, symbol moco:STSPIN32F0A
- added C1, C10, C12, C6, C9: 100nF, Capacitor_SMD:C_0402_1005Metric, symbol Device:C_Small
- added C11, C13: 1uF, Capacitor_SMD:C_0402_1005Metric, symbol Device:C_Small
- added C2, C4: 6.8pF, Capacitor_SMD:C_0402_1005Metric, symbol Device:C_Small
- added C7: 10uF, Capacitor_SMD:C_0402_1005Metric, symbol Device:C_Small
- added C8: 220nF/50V, Capacitor_SMD:C_0805_2012Metric, symbol Device:C_Small
- added C?: 10uF, Capacitor_SMD:C_0805_2012Metric, symbol Device:C
- added C?: 10uF/50V, Capacitor_SMD:C_0805_2012Metric, symbol Device:C
- added C?: 100nF, Capacitor_SMD:C_0402_1005Metric, symbol Device:C
- added D?: MBR180S1, Diode_SMD:D_SOD-123F, symbol Diode:1N6857UR
- added H? (x4): MountingHole, MountingHole:MountingHole_3.2mm_M3_ISO14580, symbol Mechanical:MountingHole
- added J?: Debug, Connector_PinHeader_2.54mm:PinHeader_2x04_P2.54mm_Vertical, symbol Connector_Generic:Conn_02x04_Odd_Even
- added J?: V+, moco:wire_rectagnel_3.7mm_D1.5mm, symbol Connector_Generic:Conn_01x01
- added J?: V-, moco:wire_circ_3.7mm_D1.5mm, symbol Connector_Generic:Conn_01x01
- added J? (x2): CAN, Connector_JST:JST_GH_SM03B-GHS-TB_1x03-1MP_P1.25mm_Horizontal, symbol Connector_Generic:Conn_01x03
- added L?: 18uH, Inductor_SMD:L_Neosid_SMS-ME3015, symbol Device:L
- added LD?: Blue, LED_SMD:LED_0603_1608Metric, symbol Device:LED
- added LD?: Red, LED_SMD:LED_0603_1608Metric, symbol Device:LED
- added R1: 120R, Resistor_SMD:R_0402_1005Metric_Pad0.72x0.64mm_HandSolder, symbol Device:R_Small
- added R4: 22k, Resistor_SMD:R_0402_1005Metric, symbol Device:R
- added R?: 1k, Resistor_SMD:R_0402_1005Metric, symbol Device:R
- added R? (x3): 10k, Resistor_SMD:R_0402_1005Metric, symbol Device:R
- added R?: 100k, Resistor_SMD:R_0402_1005Metric, symbol Device:R
- added SB1: SolderJumper_2_Open, Jumper:SolderJumper-2_P1.3mm_Open_RoundedPad1.0x1.5mm, symbol Jumper:SolderJumper_2_Open
- added SW?: RESET, Button_Switch_SMD:SW_SPST_EVQP7C, symbol Switch:SW_Push
- added TP?: GND, TestPoint:TestPoint_Pad_D1.0mm, symbol Connector:TestPoint
- added TP?: CANL, TestPoint:TestPoint_Pad_D1.0mm, symbol Connector:TestPoint
- added TP?: VCC, TestPoint:TestPoint_Pad_D1.0mm, symbol Connector:TestPoint
- added TP?: 3.3V, TestPoint:TestPoint_Pad_D1.0mm, symbol Connector:TestPoint
- added TP?: CANH, TestPoint:TestPoint_Pad_D1.0mm, symbol Connector:TestPoint
- added U1: STSPIN32G4, moco:VFQFPN 9X9X1.0 64 PITCH 0.5, symbol moco:STSPIN32G4
- added U2: TCAN337, Package_SO:SOIC-8_3.9x4.9mm_P1.27mm, symbol Interface_CAN_LIN:TCAN337
- added Y1: 16MHz, Crystal:Crystal_SMD_3225-4Pin_3.2x2.5mm, symbol Device:Crystal_GND24
- R8: LCSC (none) -> C25744; MFR. Part# (none) -> 0402WGF1002TCE
Connections:
- net +3.3V: now also C1.2, C10.2, C11.2, C12.2, C13.2, C6.2, C7.2, C9.2, J?.1 (Pin_1), R4.1, R?.2, TP?.1, U1.1 (REG3V3/VDD), U1.2 (VBAT), U1.26 (VREF+), U1.27 (VDDA), U2.3 (VCC); no longer R8.1
- net GND: now also R8.2, C1.1, C10.1, C11.1, C12.1, C13.1, C2.1, C4.1, C6.1, C7.1, C8.2, C9.1, C?.2, C?.2, C?.2, D?.2 (A), J?.1 (Pin_1), J?.2 (Pin_2), J?.2 (Pin_2), J?.2 (Pin_2), J?.8 (Pin_8), LD?.1 (K), LD?.1 (K), R?.1, SW?.2, TP?.1, U1.32 (PGND), U1.59 (PB8), U1.65 (VSS), U2.2 (GND), Y1.2, Y1.4
- net SPI_MISO: now also U1.55 (PB4)
- net SPI_MOSI: now also U1.56 (PB5)
- net ~{RESET}: now also C?.1, R?.1, SW?.1, U1.8 (PG10); no longer R8.2
- new net: D?.1 (K), L?.1, U1.62 (SW)
- new net: LD?.2 (A), R?.2 (x2)
- new net: R1.1, SB1.2 (B)
- new net CANH: J?.3 (Pin_3), J?.3 (Pin_3), SB1.1 (A), TP?.1, U2.7 (CANH)
- new net CANL: J?.1 (Pin_1), J?.1 (Pin_1), R1.2, TP?.1, U2.6 (CANL)
- new net CAN_RX: U1.47 (PA11), U2.4 (RXD)
- new net CAN_TX: U1.48 (PA12), U2.1 (TXD)
- new net OPAMP1_VINM: U1.16 (PA3)
- new net OPAMP1_VINP: U1.14 (PA1)
- new net OPAMP1_VOUT: U1.15 (PA2)
- new net OPAMP2_VINM: U1.22 (PC5)
- new net OPAMP2_VINP: U1.20 (PA7)
- new net OPAMP2_VOUT: U1.19 (PA6)
- new net OPAMP3_VINM: U1.25 (PB2)
- new net OPAMP3_VINP: U1.23 (PB0)
- new net OPAMP3_VOUT: U1.24 (PB1)
- new net OSC_IN: C2.2, U1.6 (PF0), Y1.3
- new net OSC_OUT: C4.2, U1.7 (PF1), Y1.1
- new net SCREF: R4.2, R8.1, U1.52 (SCREF)
- new net SPI_SCLK: U1.54 (PB3)
- new net SPI_~{CS}_RS: U1.57 (PB6)
- new net SWCLK: J?.5 (Pin_5), U1.50 (PA14)
- new net SWDIO: J?.3 (Pin_3), U1.49 (PA13)
- new net SWO: J?.7 (Pin_7), U1.51 (PA15)
- new net USART_RX: J?.6 (Pin_6), U1.46 (PA10)
- new net USART_TX: J?.4 (Pin_4), U1.45 (PA9)
- new net USER_LED: R?.1, U1.13 (PA0)
- new net VBUS: C8.1, C?.1, J?.1 (Pin_1), R?.2, U1.61 (VM)
- new net VCC: C?.1, L?.2, R?.1, TP?.1, U1.63 (VCC), U1.64 (REGIN)
- new net V_{BUS}_SENSE: R?.1, R?.2, U1.17 (PA4)
- no-connect marks 1 -> 19
Other:
- removed sheet CAN Bus
- removed sheet Rotary Position Sensor
- added sheet Rotary Sensor (rotary_sensor.kicad_sch)
- sheet Power Stage ports: added OPAN_A, OPAN_B, OPAN_C, OPAO_A, OPAO_B, OPAO_C, OPAP_A, OPAP_B, OPAP_C; removed none
- note added: "+10~35V. Limited by: - V_{BUS} sensing divider resistance - Capacitors max voltage (50V) - VCC buck output voltage setting"
- note added: "Buck output"
- note added: "Enable: 0.2~2.5V Disable: 2.9~3.3V 3.3V * 10/(22+10) ≈ 1V"
- note added: "LDO input"
- note added: "LDO output"
- note added: "LED"
- note added: "Main Power Input"
- note added: "Short-circuit protection"
- note added: "VCC=8, 10, 12 or 15V"
- note added: "V_{BUS} Sensing"
- note added: "V_{s_max} = 3.3V * (100+10)/10 = 36.3V"
- note removed: "V_{s_max}=3.3V*(68k+10k)/10k =25.74V"
- title: (none) -> moco-SC1
