File: hardware/moco-sp1/power_stage.kicad_sch (KiCad schematic)
At the start: 48 parts, among them J1 OUT_U, J2 OUT_V, J3 OUT_W, Q1 FDMD8240LET40, Q2 FDMD8240LET40, Q3 FDMD8240LET40, U1 STSPIN32F0A

Commit message: Update sp1 pcb
Parts:
- removed C1, C23, C26: 100nF/50V, Capacitor_SMD:C_0402_1005Metric, symbol Device:C
- removed C19, C22, C25: 220nF/50V, Capacitor_SMD:C_0402_1005Metric, symbol Device:C
- removed C2, C24, C27: 1nF, Capacitor_SMD:C_0402_1005Metric, symbol Device:C
- removed C20, C21: 10uF/50V, Capacitor_SMD:C_0805_2012Metric, symbol Device:C
- removed J1: OUT_U, moco:Conn_1x1_3.7_1.5, symbol Connector_Generic:Conn_01x01
- removed J2: OUT_V, moco:Conn_1x1_3.7_1.5, symbol Connector_Generic:Conn_01x01
- removed J3: OUT_W, moco:Conn_1x1_3.7_1.5, symbol Connector_Generic:Conn_01x01
- removed NT1, NT2, NT3, NT4, NT5, NT6: NetTie_2, NetTie:NetTie-2_SMD_Pad0.5mm, symbol Device:NetTie_2
- removed Q1, Q2, Q3: FDMD8240LET40, moco:PQFN-12, symbol moco:FDMD8240LET40
- removed R1, R15, R16, R2, R22, R23: 10R, Resistor_SMD:R_0402_1005Metric, symbol Device:R
- removed R17, R20, R24, R27, R3, R6: ${2RB}, Resistor_SMD:R_0402_1005Metric, symbol Device:R
- removed R18, R19, R25, R26, R4, R5: ${RA}, Resistor_SMD:R_0402_1005Metric, symbol Device:R
- removed R21, R28, R7: ${RB}, Resistor_SMD:R_0402_1005Metric, symbol Device:R
- removed RS1, RS2, RS3: ${RS}, Resistor_SMD:R_2512_6332Metric_Pad1.40x3.35mm_HandSolder, symbol Device:R
- removed U1: STSPIN32F0A, moco:VFQFN-48_7x7_EP2.8mm_Pitch0.5mm, symbol moco:STSPIN32F0A
- added C25: 22uF/50V, Capacitor_SMD:CP_Elec_5x5.8, symbol Device:C_Polarized
- added C? (x3): 220nF/50V, Capacitor_SMD:C_0805_2012Metric, symbol Device:C_Small
- added C? (x18): 10uF/50V, Capacitor_SMD:C_0805_2012Metric, symbol Device:C
- added C? (x3): 1nF, Capacitor_SMD:C_0402_1005Metric, symbol Device:C_Small
- added C? (x3): 100nF/50V, Capacitor_SMD:C_0402_1005Metric, symbol Device:C_Small
- added J?: B, moco:wire_rectagnel_3.7mm_D1.5mm, symbol Connector_Generic:Conn_01x01
- added J?: A, moco:wire_rectagnel_3.7mm_D1.5mm, symbol Connector_Generic:Conn_01x01
- added J?: C, moco:wire_rectagnel_3.7mm_D1.5mm, symbol Connector_Generic:Conn_01x01
- added NT? (x6): NetTie_2, NetTie:NetTie-2_SMD_Pad0.5mm, symbol Device:NetTie_2
- added Q1, Q2, Q3, Q4, Q5, Q6: SiDR390DP, Package_SO:PowerPAK_SO-8_Single, symbol moco:SiDR390DP
- added R? (x3): 20mΩ/3W, Resistor_SMD:R_2512_6332Metric, symbol Device:R
- added R? (x6): 1.78k, Resistor_SMD:R_0402_1005Metric, symbol Device:R_Small
- added R? (x6): 10R, Resistor_SMD:R_0402_1005Metric, symbol Device:R
- added R? (x3): 12k, Resistor_SMD:R_0402_1005Metric, symbol Device:R_Small
- added R? (x6): 24k, Resistor_SMD:R_0402_1005Metric, symbol Device:R_Small
- added U? (x3): STSPIN32G4, moco:VFQFPN 9X9X1.0 64 PITCH 0.5, symbol moco:STSPIN32G4
Connections:
- net +3.3V: now also R?.1, R?.1, R?.1
- net GND: now also R?.2, R?.2, R?.2
- new net: R?.1, U?.30 (GLS2)
- new net: C?.2, U?.38 (BOOT2)
- new net: R?.1, U?.40 (GHS2)
- new net: Q4.4 (G), R?.2
- new net: Q5.4 (G), R?.2
- new net: R?.1, U?.29 (GLS1)
- new net: Q2.4 (G), R?.2
- new net: Q1.4 (G), R?.2
- new net: Q3.4 (G), R?.2
- new net: R?.1, U?.31 (GLS3)
- new net: Q6.4 (G), R?.2
- new net: R?.1, U?.37 (GHS3)
- new net: C?.2, U?.41 (BOOT1)
- new net: R?.1, U?.43 (GHS1)
- new net: C?.2, U?.35 (BOOT3)
- new net GNDPWR: C25.2, C?.1, C?.1, C?.1, C?.2, C?.2, C?.2, C?.2, C?.2, C?.2, C?.2, C?.2, C?.2, C?.2, C?.2, C?.2, C?.2, C?.2, C?.2, C?.2, C?.2, C?.2, NT?.2, NT?.2, NT?.2, R?.2, R?.2, R?.2
- new net OPAN_A: C?.2, R?.1, R?.2
- new net OPAN_B: C?.2, R?.1, R?.2
- new net OPAN_C: C?.2, R?.1, R?.2
- new net OPAO_A: C?.1, R?.2
- new net OPAO_B: C?.1, R?.2
- new net OPAO_C: C?.1, R?.2
- new net OPAP_A: R?.1, R?.2, R?.2
- new net OPAP_B: R?.1, R?.2, R?.2
- new net OPAP_C: R?.1, R?.2, R?.2
- new net OUTA: C?.1, J?.1 (Pin_1), Q1.1 (S), Q1.2 (S), Q1.3 (S), Q4.5 (D), Q4.6 (D), Q4.7 (D), Q4.8 (D), U?.42 (OUT1)
- new net OUTB: C?.1, J?.1 (Pin_1), Q2.1 (S), Q2.2 (S), Q2.3 (S), Q3.5 (D), Q3.6 (D), Q3.7 (D), Q3.8 (D), U?.39 (OUT2)
- new net OUTC: C?.1, J?.1 (Pin_1), Q5.1 (S), Q5.2 (S), Q5.3 (S), Q6.5 (D), Q6.6 (D), Q6.7 (D), Q6.8 (D), U?.36 (OUT3)
- new net RSA+: NT?.1, R?.1
- new net RSA-: NT?.1, R?.1
- new net RSB+: NT?.1, R?.1
- new net RSB-: NT?.1, R?.1
- new net RSC+: NT?.1, R?.1
- new net RSC-: NT?.1, R?.1
- new net S2A: NT?.2, Q4.1 (S), Q4.2 (S), Q4.3 (S), R?.1
- new net S2B: NT?.2, Q3.1 (S), Q3.2 (S), Q3.3 (S), R?.1
- new net S2C: NT?.2, Q6.1 (S), Q6.2 (S), Q6.3 (S), R?.1
- new net VBUS: C25.1, C?.1, C?.1, C?.1, C?.1, C?.1, C?.1, C?.1, C?.1, C?.1, C?.1, C?.1, C?.1, C?.1, C?.1, C?.1, C?.1, C?.1, C?.1, C?.2, C?.2, C?.2, Q1.5 (D), Q1.6 (D), Q1.7 (D), Q1.8 (D), Q2.5 (D), Q2.6 (D), Q2.7 (D), Q2.8 (D), Q5.5 (D), Q5.6 (D), Q5.7 (D), Q5.8 (D)
Other:
- note added: "+"
- note added: "-"
- note added: "Bootstrap capacitors close to gate driver Gate resistors close to FETs"
- note added: "Bulk Capacitor"
- note added: "Gain_{max} = V_{DD}/(2*I_{max}*R_{S}) I_{max} = 12A, Gain_{max} = 6.875 Gain = R_{B}/R_{A} ≈ 6.74 Refer to ST AN5397"
- note added: "STM32 internal Op-Amp"
- note removed: "Bulk Capacitors"
- note removed: "I_{max} = SQRT(Power_{s} / R_{S}) Gain_{max} = V_{DD}/(2*I_{max}*R_{S}) Gain = R_{B}/R_{A} Refer to ST AN5397"
- note removed: "xN"
