File: hardware/moco-sp1/rotary_sensor.kicad_sch (KiCad schematic)
At the start: 2 parts, among them U3 AS5600

Commit message: Update sp1 pcb
Parts:
- removed C18: 100nF, Capacitor_SMD:C_0603_1608Metric_Pad1.08x0.95mm_HandSolder, symbol Device:C
- removed U3: AS5600, Package_SO:SOIC-8_3.9x4.9mm_P1.27mm, symbol moco:AS5600
- added C?: 1uF, Capacitor_SMD:C_0603_1608Metric_Pad1.08x0.95mm_HandSolder, symbol Device:C_Small
- added U?: MA702, Package_DFN_QFN:QFN-16-1EP_3x3mm_P0.5mm_EP1.75x1.75mm, symbol Sensor_Magnetic:MA730
Connections:
- net +3.3V: now also C?.2, U?.13 (VDD)
- net GND: now also C?.1, U?.10 (TEST), U?.17 (PAD), U?.8 (GND)
- new net A: U?.2 (A)
- new net B: U?.6 (B)
- new net MISO: U?.7 (MISO)
- new net MOSI: U?.4 (MOSI)
- new net SCLK: U?.12 (SCLK)
- new net Z: U?.3 (Z)
- new net ~{CS}: U?.5 (~{CS})
- no-connect marks 1 -> 5
Other:
- note added: "Internal pull-down: MOSI, MISO, SCLK, SSCK Internal pull-up: ~{CS}"
- note added: "SPI: - Mode: * 0 (CPOL=0, CPHA=0) or 1 (CPOL=1, CPHA=1) * Data sampled on first edge - 16-bit data frame - MSB first - ~{CS} pin active low - 25MHz clock"
- note removed: "3.3V operation"
- note removed: "DIR pin: GND -> CW VDD -> CCW"
